Commit message: fix: Getting the multi robot arm to work

File: robots/common/utils.xacro (robot description, xacro)
@@ -38,10 +38,10 @@
       <visual name="${prefix}${name}_visual">
         <geometry>
-          <mesh filename="package://${description_pkg}/meshes/robot_arms/${arm_id}/visual/${name}.dae" />
+          <mesh filename="package://${description_pkg}/meshes/robot_arms/${arm_name}/visual/${name}.dae" />
         </geometry>
       </visual>
       <collision name="${prefix}${name}_collision">
         <geometry>
-          <mesh filename="package://franka_description/meshes/robot_arms/${arm_id}/collision/${name}.stl" />
+          <mesh filename="package://franka_description/meshes/robot_arms/${arm_name}/collision/${name}.stl" />
         </geometry>
       </collision>
