Commit message: refactor: new convention for versioning

File: robots/common/franka_robot.xacro (robot description, xacro)
@@ -54,5 +54,5 @@
         <xacro:property name="ee_color" value="black" />
       </xacro:if>
-      <xacro:if value="${arm_id == 'fr3' or arm_id == 'fer' or arm_id == 'fr3v2' or arm_id == 'fr3v2.1'}">
+      <xacro:if value="${arm_id == 'fr3' or arm_id == 'fer' or arm_id == 'fr3v2' or arm_id == 'fr3v2_1'}">
         <xacro:property name="ee_color" value="white" />
       </xacro:if>

File: robots/fr3v2_1/fr3v2_1.srdf.xacro (robot description, xacro)
@@ -1,4 +1,4 @@
 <?xml version='1.0' encoding='utf-8'?>
-<robot xmlns:xacro="http://www.ros.org/wiki/xacro" name="fr3v2.1">
+<robot xmlns:xacro="http://www.ros.org/wiki/xacro" name="fr3v2_1">
   <xacro:include filename="$(find franka_description)/robots/common/franka_arm.srdf.xacro"/>
   <!--
@@ -7,5 +7,5 @@
     This argument is ignored.
   -->
-  <xacro:arg name="arm_id" default="fr3v2.1" />
+  <xacro:arg name="arm_id" default="fr3v2_1" />
   <!-- The prefix of the robot -->
   <xacro:arg name="arm_prefix" default="" />

File: robots/fr3v2_1/fr3v2_1.urdf.xacro (robot description, xacro)
@@ -1,4 +1,4 @@
 <?xml version='1.0' encoding='utf-8'?>
-<robot xmlns:xacro="http://www.ros.org/wiki/xacro" name="fr3v2.1">
+<robot xmlns:xacro="http://www.ros.org/wiki/xacro" name="fr3v2_1">
   <xacro:include filename="$(find franka_description)/robots/common/franka_robot.xacro"/>
   <!--
@@ -7,5 +7,5 @@
     This argument is ignored.
   -->
-  <xacro:arg name="arm_id" default="fr3v2.1" />
+  <xacro:arg name="arm_id" default="fr3v2_1" />
   <!-- The prefix of the robot -->
   <xacro:arg name="arm_prefix" default="" />
@@ -47,10 +47,10 @@
   <xacro:property name="prefix" value="$(arg arm_prefix)"/>
   <xacro:property name="modified_prefix" value="${prefix + '_' if prefix else ''}"/>
-  <xacro:franka_robot arm_id="fr3v2.1"
-                      joint_limits="${xacro.load_yaml('$(find franka_description)/robots/fr3v2.1/joint_limits.yaml')}"
-                      inertials="${xacro.load_yaml('$(find franka_description)/robots/fr3v2.1/inertials.yaml')}"
-                      kinematics="${xacro.load_yaml('$(find franka_description)/robots/fr3v2.1/kinematics.yaml')}"
-                      dynamics="${xacro.load_yaml('$(find franka_description)/robots/fr3v2.1/dynamics.yaml')}"
-                      accelerometer_config="${xacro.load_yaml('$(find franka_description)/robots/fr3v2.1/accelerometers.yaml')}"
+  <xacro:franka_robot arm_id="fr3v2_1"
+                      joint_limits="${xacro.load_yaml('$(find franka_description)/robots/fr3v2_1/joint_limits.yaml')}"
+                      inertials="${xacro.load_yaml('$(find franka_description)/robots/fr3v2_1/inertials.yaml')}"
+                      kinematics="${xacro.load_yaml('$(find franka_description)/robots/fr3v2_1/kinematics.yaml')}"
+                      dynamics="${xacro.load_yaml('$(find franka_description)/robots/fr3v2_1/dynamics.yaml')}"
+                      accelerometer_config="${xacro.load_yaml('$(find franka_description)/robots/fr3v2_1/accelerometers.yaml')}"
                       gazebo="$(arg gazebo)"
                       hand="$(arg hand)"

File: robots/tmrv0_2/argo_drive.xacro (robot description, xacro)
@@ -1,13 +1,14 @@
 <?xml version="1.0"?>
 <robot xmlns:xacro="http://www.ros.org/wiki/xacro" >
-  <xacro:include filename="$(find franka_description)/robots/tmr_v02/inertia.xacro" />
-  <xacro:macro name="caster_wheel" params="name parent length:='0.015' radius:='0.03' caster_joint_z:='-0.05' caster_steering_offset:='-0.035' *origin">
-    <xacro:property name="base_width" value="0.04" />
-    <xacro:property name="base_depth" value="0.03" />
-    <xacro:property name="base_height" value="0.003" />
+  <xacro:include filename="$(find franka_description)/robots/tmrv0_2/inertia.xacro" />
+  <xacro:macro name="argo_drive" params="name parent length:='0.04' radius:='0.05' offset_wheel_sign:='1' *origin">
+    <xacro:property name="base_width" value="0.17" />
+    <xacro:property name="base_depth" value="0.25" />
+    <xacro:property name="base_height" value="0.077" />
+    <xacro:property name="offset_wheel" value="0.085" />
     <xacro:property name="mass" value="0.5" />
     <link name="${name}_fixed_link" >
       <xacro:macro name="caster_base_geometry" params="xyz:='0 0 0'">
-        <origin xyz="0 0 ${-base_height/2}" />
+        <origin xyz="0 ${offset_wheel_sign*(base_depth/2 - offset_wheel)} ${base_height/2 - 0.004}" />
         <geometry>
           <box size="${base_width} ${base_depth} ${base_height}" />
@@ -21,13 +22,13 @@
       </visual>
       <inertial>
-        <origin xyz="-0.02365 0.00005 -0.03651" rpy="0 0 0"/>
-        <mass value="0.7"/>
+        <origin xyz="-0.00019 ${offset_wheel_sign*0.04522} 0.02947" rpy="0 0 0"/>
+        <mass value="11.5"/>
         <inertia
-          ixx="0.00049538079"
-          ixy="-0.00000042663"
-          ixz="0.00020926011"
-          iyy="0.00070424109"
-          iyz="-0.00000050221"
-          izz="0.00048449394"/>
+          ixx="0.07060497424"
+          ixy="-0.00025482709"
+          ixz="${offset_wheel_sign* (-0.00006283102)}"
+          iyy="0.03433835031"
+          iyz="${offset_wheel_sign*0.00249596715}"
+          izz="0.08926325955"/>
       </inertial>
     </link>
@@ -47,22 +48,23 @@
     </joint>
     <link name="${name}_link" >
-      <xacro:macro name="caster_wheel_geometry">
+      <xacro:macro name="argo_drive_geometry">
         <origin rpy="${pi/2} 0 0" />
         <geometry>
            <cylinder length="${length}" radius="${radius}" />
         </geometry>
-        <material name="orange">
-          <color rgba="1.0 0.5 0.0 1.0"/>
+        <material name="yellowish_brown">
+          <color rgba="0.8 0.6 0.2 1.0"/>
         </material>
       </xacro:macro>
       <visual>
-        <xacro:caster_wheel_geometry/>
+        <xacro:argo_drive_geometry/>
       </visual>
       <collision>
-        <xacro:caster_wheel_geometry/>
+        <xacro:argo_drive_geometry/>
       </collision>
+      <xacro:inertia-cylinder mass="${mass}" radius="${radius}" h="${length}" />
     </link>
     <joint name="${name}_joint" type="continuous">
-      <origin xyz ="${caster_steering_offset} 0 ${caster_joint_z}" rpy="0 0 0" />
+      <origin xyz ="0 0 0" rpy="0 0 0" />
       <parent link="${name}_steering_link" />
       <child  link="${name}_link" />

File: robots/tmrv0_2/caster_wheel.xacro (robot description, xacro)
@@ -1,14 +1,13 @@
 <?xml version="1.0"?>
 <robot xmlns:xacro="http://www.ros.org/wiki/xacro" >
-  <xacro:include filename="$(find franka_description)/robots/tmr_v02/inertia.xacro" />
-  <xacro:macro name="argo_drive" params="name parent length:='0.04' radius:='0.05' offset_wheel_sign:='1' *origin">
-    <xacro:property name="base_width" value="0.17" />
-    <xacro:property name="base_depth" value="0.25" />
-    <xacro:property name="base_height" value="0.077" />
-    <xacro:property name="offset_wheel" value="0.085" />
+  <xacro:include filename="$(find franka_description)/robots/tmrv0_2/inertia.xacro" />
+  <xacro:macro name="caster_wheel" params="name parent length:='0.015' radius:='0.03' caster_joint_z:='-0.05' caster_steering_offset:='-0.035' *origin">
+    <xacro:property name="base_width" value="0.04" />
+    <xacro:property name="base_depth" value="0.03" />
+    <xacro:property name="base_height" value="0.003" />
     <xacro:property name="mass" value="0.5" />
     <link name="${name}_fixed_link" >
       <xacro:macro name="caster_base_geometry" params="xyz:='0 0 0'">
-        <origin xyz="0 ${offset_wheel_sign*(base_depth/2 - offset_wheel)} ${base_height/2 - 0.004}" />
+        <origin xyz="0 0 ${-base_height/2}" />
         <geometry>
           <box size="${base_width} ${base_depth} ${base_height}" />
@@ -22,13 +21,13 @@
       </visual>
       <inertial>
-        <origin xyz="-0.00019 ${offset_wheel_sign*0.04522} 0.02947" rpy="0 0 0"/>
-        <mass value="11.5"/>
+        <origin xyz="-0.02365 0.00005 -0.03651" rpy="0 0 0"/>
+        <mass value="0.7"/>
         <inertia
-          ixx="0.07060497424"
-          ixy="-0.00025482709"
-          ixz="${offset_wheel_sign* (-0.00006283102)}"
-          iyy="0.03433835031"
-          iyz="${offset_wheel_sign*0.00249596715}"
-          izz="0.08926325955"/>
+          ixx="0.00049538079"
+          ixy="-0.00000042663"
+          ixz="0.00020926011"
+          iyy="0.00070424109"
+          iyz="-0.00000050221"
+          izz="0.00048449394"/>
       </inertial>
     </link>
@@ -48,23 +47,22 @@
     </joint>
     <link name="${name}_link" >
-      <xacro:macro name="argo_drive_geometry">
+      <xacro:macro name="caster_wheel_geometry">
         <origin rpy="${pi/2} 0 0" />
         <geometry>
            <cylinder length="${length}" radius="${radius}" />
         </geometry>
-        <material name="yellowish_brown">
-          <color rgba="0.8 0.6 0.2 1.0"/>
+        <material name="orange">
+          <color rgba="1.0 0.5 0.0 1.0"/>
         </material>
       </xacro:macro>
       <visual>
-        <xacro:argo_drive_geometry/>
+        <xacro:caster_wheel_geometry/>
       </visual>
       <collision>
-        <xacro:argo_drive_geometry/>
+        <xacro:caster_wheel_geometry/>
       </collision>
-      <xacro:inertia-cylinder mass="${mass}" radius="${radius}" h="${length}" />
     </link>
     <joint name="${name}_joint" type="continuous">
-      <origin xyz ="0 0 0" rpy="0 0 0" />
+      <origin xyz ="${caster_steering_offset} 0 ${caster_joint_z}" rpy="0 0 0" />
       <parent link="${name}_steering_link" />
       <child  link="${name}_link" />

File: robots/tmrv0_2/lidar.xacro (robot description, xacro)
@@ -2,5 +2,5 @@
 <robot xmlns:xacro="http://www.ros.org/wiki/xacro" >
   <xacro:macro name="lidar" params="name parent min_angle:='${radians(-45)}' max_angle:='${radians(225)}' *origin ">
-    <xacro:include filename="$(find franka_description)/robots/tmr_v02/nanoscan3/nanoscan3/nanoscan3_macro.xacro"/>
+    <xacro:include filename="$(find franka_description)/robots/tmrv0_2/nanoscan3/nanoscan3/nanoscan3_macro.xacro"/>
     <xacro:nanoscan3
       name="${name}"

File: robots/tmrv0_2/nanoscan3/nanoscan3.urdf.xacro (robot description, xacro)
@@ -8,5 +8,5 @@
   <!-- Load robot's macro with parameters -->
   <!-- set prefix if multiple robots are used -->
-  <xacro:include filename="$(find sick_safetyscanners2)/description/robots/tmr_v02/nanoscan3/nanoscan3_macro.xacro"/>
+  <xacro:include filename="$(find sick_safetyscanners2)/description/robots/tmrv0_2/nanoscan3/nanoscan3_macro.xacro"/>
   <xacro:property name="mounting_kit" value="$(arg mounting_kit)"/>
   <xacro:nanoscan3

File: robots/tmrv0_2/nanoscan3/nanoscan3/nanoscan3_macro.xacro (robot description, xacro)
@@ -1,6 +1,6 @@
 <?xml version="1.0" encoding="UTF-8"?>
 <robot xmlns:xacro="http://wiki.ros.org/xacro">
-  <xacro:include filename="$(find franka_description)/robots/tmr_v02/nanoscan3/common.xacro" />
-  <xacro:include filename="$(find franka_description)/robots/tmr_v02/nanoscan3/nanoscan3/gazebo_macro.xacro" />
+  <xacro:include filename="$(find franka_description)/robots/tmrv0_2/nanoscan3/common.xacro" />
+  <xacro:include filename="$(find franka_description)/robots/tmrv0_2/nanoscan3/nanoscan3/gazebo_macro.xacro" />
   <!-- joint offsets when mounted on frame -->
   <xacro:property name="base_x" value="0.0803"/>

File: robots/tmrv0_2/rocker_arm.xacro (robot description, xacro)
@@ -1,5 +1,5 @@
 <?xml version="1.0"?>
 <robot xmlns:xacro="http://www.ros.org/wiki/xacro" >
-  <xacro:include filename="$(find franka_description)/robots/tmr_v02/inertia.xacro" />
+  <xacro:include filename="$(find franka_description)/robots/tmrv0_2/inertia.xacro" />
   <xacro:macro name="rocker_arm" params="name mass parent *origin">
     <xacro:property name="depth" value="0.32"/>

File: robots/tmrv0_2/tmrv0_2.ros2_control.xacro (robot description, xacro)
@@ -1,5 +1,5 @@
 <?xml version="1.0"?>
 <robot xmlns:xacro="http://www.ros.org/wiki/xacro">
-  <xacro:macro name="tmr_v02_ros2_control"
+  <xacro:macro name="tmrv0_2_ros2_control"
     params="mobile_robot_id
             robot_ip
@@ -10,5 +10,5 @@
         <param name="version">0.1.0</param>
         <param name="mobile_robot_id">${mobile_robot_id}</param>
-        <param name="arm_id">tmr_v02</param>
+        <param name="arm_id">tmrv0_2</param>
         <xacro:if value="${use_fake_hardware}">
           <plugin>fake_components/GenericSystem</plugin>

File: robots/tmrv0_2/tmrv0_2.urdf.xacro (robot description, xacro)
@@ -1,5 +1,5 @@
 <?xml version='1.0' encoding='utf-8'?>
-<robot xmlns:xacro="http://www.ros.org/wiki/xacro" name="tmr_v02">
-<xacro:include filename="$(find franka_description)/robots/tmr_v02/tmr_v02.xacro"/>
+<robot xmlns:xacro="http://www.ros.org/wiki/xacro" name="tmrv0_2">
+<xacro:include filename="$(find franka_description)/robots/tmrv0_2/tmrv0_2.xacro"/>
   <!--
     DEPRECATION NOTICE
@@ -8,5 +8,5 @@
   -->
   <!-- Define arguments -->
-  <xacro:arg name="arm_id" default="tmr_v02" />
+  <xacro:arg name="arm_id" default="tmrv0_2" />
   <!-- Is the robot being controlled with ros2_control?" -->
   <xacro:arg name="ros2_control" default="false" />
@@ -26,5 +26,5 @@
     <origin rpy="0 0 0" xyz="0 0 0"/>
   </joint>
-  <xacro:tmr_v02 mobile_robot_id="$(arg arm_id)"
+  <xacro:tmrv0_2 mobile_robot_id="$(arg arm_id)"
               robot_ip="$(arg robot_ip)"
               ros2_control="$(arg ros2_control)"

File: robots/tmrv0_2/tmrv0_2.xacro (robot description, xacro)
@@ -1,5 +1,5 @@
 <?xml version="1.0"?>
 <robot xmlns:xacro="http://www.ros.org/wiki/xacro">
-  <xacro:macro name="tmr_v02"
+  <xacro:macro name="tmrv0_2"
     params="mobile_robot_id
                   robot_ip:=''
@@ -8,9 +8,9 @@
                   fake_sensor_commands:=false
                   reduced_version:=false">
-    <xacro:include filename="$(find franka_description)/robots/tmr_v02/argo_drive.xacro" />
-    <xacro:include filename="$(find franka_description)/robots/tmr_v02/caster_wheel.xacro" />
-    <xacro:include filename="$(find franka_description)/robots/tmr_v02/rocker_arm.xacro" />
-    <xacro:include filename="$(find franka_description)/robots/tmr_v02/inertia.xacro" />
-    <xacro:include filename="$(find franka_description)/robots/tmr_v02/lidar.xacro" />
+    <xacro:include filename="$(find franka_description)/robots/tmrv0_2/argo_drive.xacro" />
+    <xacro:include filename="$(find franka_description)/robots/tmrv0_2/caster_wheel.xacro" />
+    <xacro:include filename="$(find franka_description)/robots/tmrv0_2/rocker_arm.xacro" />
+    <xacro:include filename="$(find franka_description)/robots/tmrv0_2/inertia.xacro" />
+    <xacro:include filename="$(find franka_description)/robots/tmrv0_2/lidar.xacro" />
     <xacro:property name="caster_radius" value="0.03" />
     <xacro:property name="caster_x" value="0.3" />
@@ -34,5 +34,5 @@
         <origin xyz="0 0 0" rpy="0 0 ${pi}" />
         <geometry>
-          <mesh filename="package://franka_description/meshes/tmr_v02/visual/tmr_v02.stl" />
+          <mesh filename="package://franka_description/meshes/tmrv0_2/visual/tmrv0_2.stl" />
         </geometry>
         <material name="white">
@@ -43,5 +43,5 @@
         <origin xyz="0 0 0" rpy="0 0 ${pi}" />
         <geometry>
-          <mesh filename="package://franka_description/meshes/tmr_v02/collision/tmr_v02.stl" />
+          <mesh filename="package://franka_description/meshes/tmrv0_2/collision/tmrv0_2.stl" />
         </geometry>
       </collision>
@@ -136,6 +136,6 @@
     </joint>
     <xacro:if value="${ros2_control}">
-      <xacro:include filename="$(find franka_description)/robots/tmr_v02/tmr_v02.ros2_control.xacro" />
-      <xacro:tmr_v02_ros2_control
+      <xacro:include filename="$(find franka_description)/robots/tmrv0_2/tmrv0_2.ros2_control.xacro" />
+      <xacro:tmrv0_2_ros2_control
         mobile_robot_id="${mobile_robot_id}"
         robot_ip="${robot_ip}"
