Commit message: feat: Added the tmr description

File: robots/common/franka_arm.ros2_control.xacro (robot description, xacro)
@@ -62,4 +62,5 @@
         <xacro:configure_joint joint_name="${arm_prefix}${arm_id}_finger_joint1" initial_position="0.0" />
       </xacro:if>
+      <!-- General purpose IO interfaces -->
       <xacro:macro name="general_purpose_io" params="prefix command_interface index">
         <gpio name="${prefix}">
@@ -69,14 +70,15 @@
       </xacro:macro>
       <!-- Cartesian velocity interfaces -->
-      <xacro:general_purpose_io prefix="vx" command_interface="cartesian_velocity" index="0"/>
-      <xacro:general_purpose_io prefix="vy" command_interface="cartesian_velocity" index="1"/>
-      <xacro:general_purpose_io prefix="vz" command_interface="cartesian_velocity" index="2"/>
-      <xacro:general_purpose_io prefix="wx" command_interface="cartesian_velocity" index="3"/>
-      <xacro:general_purpose_io prefix="wy" command_interface="cartesian_velocity" index="4"/>
-      <xacro:general_purpose_io prefix="wz" command_interface="cartesian_velocity" index="5"/>
+      <xacro:property name="gpios_suffix" value="${'' if arm_prefix == '' else arm_prefix_modified + arm_id + '_'}" />
+      <xacro:general_purpose_io prefix="${gpios_suffix}vx" command_interface="cartesian_velocity" index="0"/>
+      <xacro:general_purpose_io prefix="${gpios_suffix}vy" command_interface="cartesian_velocity" index="1"/>
+      <xacro:general_purpose_io prefix="${gpios_suffix}vz" command_interface="cartesian_velocity" index="2"/>
+      <xacro:general_purpose_io prefix="${gpios_suffix}wx" command_interface="cartesian_velocity" index="3"/>
+      <xacro:general_purpose_io prefix="${gpios_suffix}wy" command_interface="cartesian_velocity" index="4"/>
+      <xacro:general_purpose_io prefix="${gpios_suffix}wz" command_interface="cartesian_velocity" index="5"/>
       <!-- Cartesian pose interfaces, in total 16 interfaces -->
       <xacro:macro name="loop" params="i">
         <xacro:unless value="${i == 16}">
-          <xacro:general_purpose_io prefix="${i}" command_interface="cartesian_pose_command" index="${i}"/>
+          <xacro:general_purpose_io prefix="${gpios_suffix}${i}" command_interface="cartesian_pose_command" index="${i}"/>
           <xacro:loop i="${i+1}"/>
         </xacro:unless>
@@ -84,6 +86,6 @@
       <xacro:loop i="0"/>
       <!-- Elbow command interfaces -->
-      <xacro:general_purpose_io prefix="joint_3_position" command_interface="elbow_command" index="0"/>
-      <xacro:general_purpose_io prefix="joint_4_sign" command_interface="elbow_command" index="1"/>
+      <xacro:general_purpose_io prefix="${gpios_suffix}joint_3_position" command_interface="elbow_command" index="0"/>
+      <xacro:general_purpose_io prefix="${gpios_suffix}joint_4_sign" command_interface="elbow_command" index="1"/>
     </ros2_control>
     <xacro:if value="${gazebo}">

Commit message: refactor: tmr branch working with jazzy

File: robots/common/franka_arm.ros2_control.xacro (robot description, xacro)
@@ -9,6 +9,5 @@
                  hand:=false
                  gazebo_effort:=false
-                 arm_prefix:=''
-                 multi_arm:=false">
+                 arm_prefix:=''">
     <xacro:property name="arm_prefix_modified" value="${'' if arm_prefix == '' else arm_prefix + '_'}" />
     <ros2_control name="${arm_prefix_modified}FrankaHardwareInterface" type="system">

File: robots/common/utils.xacro (robot description, xacro)
@@ -38,10 +38,10 @@
       <visual name="${prefix}${name}_visual">
         <geometry>
-          <mesh filename="package://${description_pkg}/meshes/robot_arms/${arm_name}/visual/${name}.dae" />
+          <mesh filename="package://${description_pkg}/meshes/robot_arms/${arm_id}/visual/${name}.dae" />
         </geometry>
       </visual>
       <collision name="${prefix}${name}_collision">
         <geometry>
-          <mesh filename="package://franka_description/meshes/robot_arms/${arm_name}/collision/${name}.stl" />
+          <mesh filename="package://franka_description/meshes/robot_arms/${arm_id}/collision/${name}.stl" />
         </geometry>
       </collision>

File: robots/multi_arm/multi_arm.urdf.xacro (robot description, xacro)
@@ -117,6 +117,5 @@
                             no_prefix="$(arg no_prefix)"
                             arm_prefix= "${arm_prefixes_list[i]}"
-                            connected_to="${arm_prefixes_list[i]}_base"
-                            multi_arm="$(arg multi_arm)">
+                            connected_to="${arm_prefixes_list[i]}_base">
         </xacro:franka_robot>
       </xacro:unless>

Commit message: chore: tmr v02 files renamed

File: robots/common/franka_arm.ros2_control.xacro (robot description, xacro)
@@ -61,5 +61,4 @@
         <xacro:configure_joint joint_name="${arm_prefix}${arm_id}_finger_joint1" initial_position="0.0" />
       </xacro:if>
-      <!-- General purpose IO interfaces -->
       <xacro:macro name="general_purpose_io" params="prefix command_interface index">
         <gpio name="${prefix}">
@@ -69,15 +68,14 @@
       </xacro:macro>
       <!-- Cartesian velocity interfaces -->
-      <xacro:property name="gpios_suffix" value="${'' if arm_prefix == '' else arm_prefix_modified + arm_id + '_'}" />
-      <xacro:general_purpose_io prefix="${gpios_suffix}vx" command_interface="cartesian_velocity" index="0"/>
-      <xacro:general_purpose_io prefix="${gpios_suffix}vy" command_interface="cartesian_velocity" index="1"/>
-      <xacro:general_purpose_io prefix="${gpios_suffix}vz" command_interface="cartesian_velocity" index="2"/>
-      <xacro:general_purpose_io prefix="${gpios_suffix}wx" command_interface="cartesian_velocity" index="3"/>
-      <xacro:general_purpose_io prefix="${gpios_suffix}wy" command_interface="cartesian_velocity" index="4"/>
-      <xacro:general_purpose_io prefix="${gpios_suffix}wz" command_interface="cartesian_velocity" index="5"/>
+      <xacro:general_purpose_io prefix="vx" command_interface="cartesian_velocity" index="0"/>
+      <xacro:general_purpose_io prefix="vy" command_interface="cartesian_velocity" index="1"/>
+      <xacro:general_purpose_io prefix="vz" command_interface="cartesian_velocity" index="2"/>
+      <xacro:general_purpose_io prefix="wx" command_interface="cartesian_velocity" index="3"/>
+      <xacro:general_purpose_io prefix="wy" command_interface="cartesian_velocity" index="4"/>
+      <xacro:general_purpose_io prefix="wz" command_interface="cartesian_velocity" index="5"/>
       <!-- Cartesian pose interfaces, in total 16 interfaces -->
       <xacro:macro name="loop" params="i">
         <xacro:unless value="${i == 16}">
-          <xacro:general_purpose_io prefix="${gpios_suffix}${i}" command_interface="cartesian_pose_command" index="${i}"/>
+          <xacro:general_purpose_io prefix="${i}" command_interface="cartesian_pose_command" index="${i}"/>
           <xacro:loop i="${i+1}"/>
         </xacro:unless>
@@ -85,6 +83,6 @@
       <xacro:loop i="0"/>
       <!-- Elbow command interfaces -->
-      <xacro:general_purpose_io prefix="${gpios_suffix}joint_3_position" command_interface="elbow_command" index="0"/>
-      <xacro:general_purpose_io prefix="${gpios_suffix}joint_4_sign" command_interface="elbow_command" index="1"/>
+      <xacro:general_purpose_io prefix="joint_3_position" command_interface="elbow_command" index="0"/>
+      <xacro:general_purpose_io prefix="joint_4_sign" command_interface="elbow_command" index="1"/>
     </ros2_control>
     <xacro:if value="${gazebo}">

Commit message: feat: pass async feature

File: robots/common/franka_arm.ros2_control.xacro (robot description, xacro)
@@ -9,12 +9,14 @@
                  hand:=false
                  gazebo_effort:=false
-                 arm_prefix:=''">
-    <xacro:property name="arm_prefix_modified" value="${'' if arm_prefix == '' else arm_prefix + '_'}" />
-    <ros2_control name="${arm_prefix_modified}FrankaHardwareInterface" type="system" is_async="true">
-        <properties>
-          <async scheduling_policy="detached" print_warnings="false"/>
-        </properties>
+                 arm_prefix:=''
+                 is_async:=false">
+    <ros2_control name="${arm_prefix}FrankaHardwareInterface" type="system" is_async="${is_async}">
+        <xacro:if value="${is_async}">
+          <properties>
+            <async scheduling_policy="detached" print_warnings="true" thread_priority="99" manage_overruns="false"/>
+          </properties>
+        </xacro:if>
         <hardware>
-          <param name="version">0.1.0</param>
+          <param name="version">1.0.0</param>
           <param name="robot_type">${robot_type}</param>
           <param name="prefix">${arm_prefix}</param>

File: robots/common/franka_robot.xacro (robot description, xacro)
@@ -29,5 +29,6 @@
                       arm_prefix:=''
                       description_pkg:='franka_description'
-                      connected_to:='base'">
+                      connected_to:='base'
+                      is_async:=false">
     <xacro:include filename="$(find franka_description)/robots/common/utils.xacro" />
     <xacro:include filename="$(find franka_description)/robots/common/franka_arm.xacro" />
@@ -152,4 +153,5 @@
           gazebo_effort="${gazebo_effort}"
           arm_prefix="${arm_prefix}"
+          is_async="${is_async}"
       />
     </xacro:if>

File: robots/fr3_duo/fr3_duo.urdf.xacro (robot description, xacro)
@@ -42,4 +42,6 @@
   <!-- Name of the description package -->
   <xacro:arg name="description_pkg" default="franka_description" />
+  <!-- Are the robots using the async hardware interface? -->
+  <xacro:arg name="is_async" default="false" />
   <link name="base">
   </link>
@@ -96,5 +98,6 @@
                           arm_prefix= "${modified_prefix}"
                           description_pkg="$(arg description_pkg)"
-                          connected_to="${arm_prefixes_list[i]}_base">
+                          connected_to="${arm_prefixes_list[i]}_base"
+                          is_async="$(arg is_async)">
       </xacro:franka_robot>
       <xacro:loop i="${i+1}"/>
