Commit message: feat: torso added to the description

File: robots/multi_arm/multi_arm.urdf.xacro (robot description, xacro)
@@ -8,12 +8,12 @@
   -->
   <!-- Define arguments -->
-  <xacro:arg name="arm_ids" default="['fr3','fr3']" />
+  <xacro:arg name="arm_ids" default="['fr3','fr3','tmr']" />
   <xacro:property name="arm_ids_list" value="${$(arg arm_ids)}" />
-  <xacro:arg name="number_of_robots" default = "2"/>
+  <xacro:arg name="number_of_robots" default = "3"/>
   <!-- Define arguments -->
-  <xacro:arg name="xyz_values" default="['0 0.1 0','0 -0.1 0']" />
+  <xacro:arg name="xyz_values" default="['0.15 0.05 0.65','0.15 -0.05 0.65','0 0 0']" />
   <xacro:property name="xyz_list" value="${$(arg xyz_values)}" />
   <!-- Define arguments -->
-  <xacro:arg name="rpy_values" default="['-0.7 0 0','0.7 0 0']" />
+  <xacro:arg name="rpy_values" default="['-0.89334809 -0.17456074 -0.46334506','0.89334809 -0.17456074 0.46334506','0 0 0']" />
   <xacro:property name="rpy_list" value="${$(arg rpy_values)}" />
   <!-- Don't print a prefix for joints, visuals, and links? -->
@@ -28,5 +28,5 @@
   <xacro:arg name="ros2_control" default="false" />
   <!-- IP address or hostname of the robot" -->
-  <xacro:arg name="robot_ips" default="['172.16.0.2','172.16.0.3']" />
+  <xacro:arg name="robot_ips" default="['172.16.0.2','172.16.0.3', '172.16.0.4']" />
   <xacro:property name="robot_ips_list" value="${$(arg robot_ips)}" />
   <!-- Should a fake hardware be used? -->
@@ -40,10 +40,21 @@
   <!-- Prefixes for arm -->
   <!-- TODO: check if the list size is correct -->
-  <xacro:arg name="arm_prefixes" default="['left','right']" />
+  <xacro:arg name="arm_prefixes" default="['left','right','platform']" />
   <xacro:property name="arm_prefixes_list" value="${$(arg arm_prefixes)}" />
   <!-- For a multi arm setup, we need a threaded robot running async-->
   <xacro:arg name="multi_arm" default="true" />
+  <!-- Flag to use the torso if two arms are used-->
+  <xacro:arg name="use_torso" default="true" />
+  <xacro:property name="use_torso_flag" value="$(arg use_torso)"/>
   <link name="base">
   </link>
+  <!-- torso -->
+  <xacro:if value="${use_torso_flag}">
+    <xacro:include filename="$(find franka_description)/extras/torso_duo/torso.xacro"/>
+    <xacro:arg name="torso_kinematics" default="$(find franka_description)/extras/torso_duo/kinematics.yaml"/>
+    <xacro:torso name="torso" parent="base_link">
+      <origin xyz="0.20 0 0.30" rpy="0 0 0" />
+    </xacro:torso>
+  </xacro:if>
   <!-- The multi robot setup configures 'multi_arm' by default to true s.t. it uses the async threading approach for the hardware interface -->
   <xacro:include filename="$(find franka_description)/robots/tmr.xacro"/>
@@ -63,9 +74,26 @@
       </xacro:if>
       <xacro:unless value="${arm_ids_list[i] == 'tmr'}">
-        <joint name="${arm_prefixes_list[i]}_base_joint" type="fixed">
-          <parent link="base"/>
-          <child link="${arm_prefixes_list[i]}_base"/>
-          <origin rpy="${rpy_list[i]}" xyz="${xyz_list[i]}"/>
-        </joint>
+        <xacro:unless value="${use_torso_flag}">
+          <joint name="${arm_prefixes_list[i]}_base_joint" type="fixed">
+            <parent link="base"/>
+            <child link="${arm_prefixes_list[i]}_base"/>
+            <origin rpy="${rpy_list[i]}" xyz="${xyz_list[i]}"/>
+          </joint>
+        </xacro:unless>
+        <xacro:if value="${use_torso_flag}">
+          <xacro:property name="torso_to_base" value="${xacro.load_yaml('$(arg torso_kinematics)')}"/>
+          <xacro:property name="robot_prefix" value="${arm_prefixes_list[i]}"/>
+          <joint name="${arm_prefixes_list[i]}_base_joint" type="fixed">
+            <parent link="torso_link"/>
+            <child link="${arm_prefixes_list[i]}_base"/>
+            <xacro:if value="${robot_prefix == 'left'}">
+              <xacro:property name="torso_corner" value="${torso_to_base['left']}" lazy_eval="false" />
+            </xacro:if>
+            <xacro:if value="${robot_prefix == 'right'}">
+              <xacro:property name="torso_corner" value="${torso_to_base['right']}" lazy_eval="false" />
+            </xacro:if>
+            <origin rpy="${torso_corner.kinematic.roll} ${torso_corner.kinematic.pitch} ${torso_corner.kinematic.yaw}" xyz="${torso_corner.kinematic.x} ${torso_corner.kinematic.y} ${torso_corner.kinematic.z}"/>
+          </joint>
+        </xacro:if>
       <xacro:property name="arm_id_i" value="${arm_ids_list[i]}"/>
       <xacro:arg name="inertials_path" default="$(find franka_description)/robots/${arm_id_i}/inertials.yaml"/>

Commit message: refactor: tmr related files are placed in dedicated folders

File: robots/multi_arm/multi_arm.urdf.xacro (robot description, xacro)
@@ -58,5 +58,5 @@
   </xacro:if>
   <!-- The multi robot setup configures 'multi_arm' by default to true s.t. it uses the async threading approach for the hardware interface -->
-  <xacro:include filename="$(find franka_description)/robots/tmr.xacro"/>
+  <xacro:include filename="$(find franka_description)/robots/tmr/tmr.xacro"/>
   <xacro:macro name="loop" params="i">
     <xacro:unless value="${i == $(arg number_of_robots)}">

File: robots/tmr/bogie.xacro (robot description, xacro)
@@ -1,5 +1,5 @@
 <?xml version="1.0"?>
 <robot xmlns:xacro="http://www.ros.org/wiki/xacro" >
-  <xacro:include filename="$(find franka_description)/robots/inertia.xacro" />
+  <xacro:include filename="$(find franka_description)/robots/tmr/inertia.xacro" />
   <xacro:macro name="bogie" params="name mass parent *origin">
     <xacro:property name="depth" value="0.32"/>

File: robots/tmr/caster_wheel.urdf.xacro (robot description, xacro)
@@ -1,5 +1,5 @@
 <?xml version="1.0"?>
 <robot name="caster" xmlns:xacro="http://www.ros.org/wiki/xacro" >
-  <xacro:include filename="$(find franka_description)/robots/caster_wheel.xacro" />
+  <xacro:include filename="$(find franka_description)/robots/tmr/caster_wheel.xacro" />
   <link name="world" />
   <xacro:caster_wheel name="caster" mass="0.3" radius="0.05" length="0.02" parent="world" caster_joint_z="-0.08" caster_steering_offset="-0.04">

File: robots/tmr/caster_wheel.xacro (robot description, xacro)
@@ -1,5 +1,5 @@
 <?xml version="1.0"?>
 <robot xmlns:xacro="http://www.ros.org/wiki/xacro" >
-  <xacro:include filename="$(find franka_description)/robots/inertia.xacro" />
+  <xacro:include filename="$(find franka_description)/robots/tmr/inertia.xacro" />
   <xacro:macro name="caster_wheel" params="name mass parent length:='0.025' radius:='0.05' caster_joint_z:='-0.074' caster_steering_offset:='-0.035' *origin">
     <xacro:property name="base_width" value="0.04" />
@@ -33,5 +33,5 @@
         <origin rpy="${pi/2} 0 ${pi/2}" />
         <geometry>
-           <mesh filename="package://franka_description/meshes/visual/caster.stl"/>
+           <mesh filename="package://franka_description/meshes/tmr/visual/caster.stl"/>
         </geometry>
         <material name="darkgrey">

File: robots/tmr/inertia.xacro (robot description, xacro)
@@ -31,4 +31,13 @@
     </inertial>
   </xacro:macro>
+  <xacro:macro name="inertia-torso">
+    <inertial>
+      <origin xyz="-0.374101 0.001522 0.120542" rpy="0 0 0" />
+      <mass value="75.711368" />
+      <inertia  ixx ="1.822241406454"	ixy ="0.009367998445"	ixz ="0.855091055826"
+	              iyx ="0.009367998445"	iyy ="4.242134556907"	iyz ="-0.012022054390"
+	              izx ="0.855091055826"	izy ="-0.012022054390" izz ="4.568496104964"/>
+    </inertial>
+  </xacro:macro>
   <xacro:macro name="inertia-default" params="mass">
     <inertial>

File: robots/tmr/lidar.xacro (robot description, xacro)
@@ -2,5 +2,5 @@
 <robot xmlns:xacro="http://www.ros.org/wiki/xacro" >
   <xacro:macro name="lidar" params="name parent min_angle:='${radians(-45)}' max_angle:='${radians(225)}' *origin ">
-    <xacro:include filename="$(find franka_description)/robots/nanoscan3/nanoscan3/nanoscan3_macro.xacro"/>
+    <xacro:include filename="$(find franka_description)/robots/tmr/nanoscan3/nanoscan3/nanoscan3_macro.xacro"/>
     <xacro:nanoscan3
       name="${name}"

File: robots/tmr/nanoscan3/nanoscan3.urdf.xacro (robot description, xacro)
@@ -8,5 +8,5 @@
   <!-- Load robot's macro with parameters -->
   <!-- set prefix if multiple robots are used -->
-  <xacro:include filename="$(find sick_safetyscanners2)/description/robots/nanoscan3/nanoscan3_macro.xacro"/>
+  <xacro:include filename="$(find sick_safetyscanners2)/description/robots/tmr/nanoscan3/nanoscan3_macro.xacro"/>
   <xacro:property name="mounting_kit" value="$(arg mounting_kit)"/>
   <xacro:nanoscan3

File: robots/tmr/nanoscan3/nanoscan3/nanoscan3_macro.xacro (robot description, xacro)
@@ -1,6 +1,6 @@
 <?xml version="1.0" encoding="UTF-8"?>
 <robot xmlns:xacro="http://wiki.ros.org/xacro">
-  <xacro:include filename="$(find franka_description)/robots/nanoscan3/common.xacro" />
-  <xacro:include filename="$(find franka_description)/robots/nanoscan3/nanoscan3/gazebo_macro.xacro" />
+  <xacro:include filename="$(find franka_description)/robots/tmr/nanoscan3/common.xacro" />
+  <xacro:include filename="$(find franka_description)/robots/tmr/nanoscan3/nanoscan3/gazebo_macro.xacro" />
   <!-- joint offsets when mounted on frame -->
   <xacro:property name="base_x" value="0.0803"/>

File: robots/tmr/tmr.urdf.xacro (robot description, xacro)
@@ -11,5 +11,5 @@
   <!-- Should fake sensors be used? -->
   <xacro:arg name="fake_sensor_commands" default="false" />
-  <xacro:include filename="$(find franka_description)/robots/tmr.xacro" />
+  <xacro:include filename="$(find franka_description)/robots/tmr/tmr.xacro" />
   <xacro:tmr
     mobile_robot_id="$(arg mobile_robot_id)"

File: robots/tmr/tmr.xacro (robot description, xacro)
@@ -7,11 +7,10 @@
                   use_fake_hardware:=false
                   fake_sensor_commands:=false">
-    <xacro:include filename="$(find franka_description)/robots/wheel.xacro" />
-    <xacro:include filename="$(find franka_description)/robots/caster_wheel.xacro" />
-    <xacro:include filename="$(find franka_description)/robots/bogie.xacro" />
-    <xacro:include filename="$(find franka_description)/robots/inertia.xacro" />
-    <xacro:include filename="$(find franka_description)/robots/lidar.xacro" />
+    <xacro:include filename="$(find franka_description)/robots/tmr/wheel.xacro" />
+    <xacro:include filename="$(find franka_description)/robots/tmr/caster_wheel.xacro" />
+    <xacro:include filename="$(find franka_description)/robots/tmr/bogie.xacro" />
+    <xacro:include filename="$(find franka_description)/robots/tmr/inertia.xacro" />
+    <xacro:include filename="$(find franka_description)/robots/tmr/lidar.xacro" />
     <xacro:include filename="$(find realsense2_description)/urdf/_d455.urdf.xacro" />
-    <xacro:include filename="$(find olv_module_descriptions)/urdf/olv-imu01.urdf.xacro" />
     <xacro:property name="caster_radius" value="0.05" />
     <xacro:property name="caster_mass" value="0.5" />
@@ -43,5 +42,5 @@
         <origin xyz="0 0 0" rpy="0 0 ${pi}" />
         <geometry>
-          <mesh filename="package://franka_description/meshes/visual/tmr_base.dae" />
+          <mesh filename="package://franka_description/meshes/tmr/visual/tmr_base.dae" />
         </geometry>
         <material name="white">
@@ -52,5 +51,5 @@
         <origin xyz="0 0 0" rpy="0 0 ${pi}" />
         <geometry>
-          <mesh filename="package://franka_description/meshes/collision/tmr_base_simplified.stl" />
+          <mesh filename="package://franka_description/meshes/tmr/collision/tmr_base_simplified.stl" />
         </geometry>
       </collision>
@@ -121,5 +120,5 @@
     </xacro:sensor_d455>
     <xacro:if value="${ros2_control}">
-      <xacro:include filename="$(find franka_description)/robots/tmr.ros2_control.xacro" />
+      <xacro:include filename="$(find franka_description)/robots/tmr/tmr.ros2_control.xacro" />
       <xacro:tmr_ros2_control
         mobile_robot_id="${mobile_robot_id}"
@@ -129,14 +128,4 @@
       />
     </xacro:if>
-   <!-- IMU -->
-   <link name="imu">
-    </link>
-    <joint name="base_to_imu" type="fixed">
-      <parent link="base_link"/>
-      <child link="imu"/>
-      <origin xyz="-0.176 0.0545 0.15" rpy="${pi/2} 0 ${-pi/2}"/>
-    </joint>
-   <xacro:olv-imu01 namespace="olv-imu01" parent_link="imu" mounting_side="bottom" mounting_rotation="0" >
-   </xacro:olv-imu01>
   </xacro:macro>
 </robot>

File: robots/tmr/wheel.urdf.xacro (robot description, xacro)
@@ -1,5 +1,5 @@
 <?xml version="1.0"?>
 <robot name="wheel" xmlns:xacro="http://www.ros.org/wiki/xacro" >
-  <xacro:include filename="$(find franka_description)/robots/wheel.xacro" />
+  <xacro:include filename="$(find franka_description)/robots/tmr/wheel.xacro" />
   <link name="world" />
   <xacro:wheel lr="left" mass="3" parent="world" radius="0.125" wheel_width="0.06">

File: robots/tmr/wheel.xacro (robot description, xacro)
@@ -1,5 +1,5 @@
 <?xml version="1.0"?>
 <robot xmlns:xacro="http://www.ros.org/wiki/xacro" >
-  <xacro:include filename="$(find franka_description)/robots/inertia.xacro" />
+  <xacro:include filename="$(find franka_description)/robots/tmr/inertia.xacro" />
   <xacro:macro name="wheel" params="lr mass parent radius:='0.125' wheel_width:='0.06' *origin">
     <link name="${lr[0]}_wheel_link" >
@@ -12,5 +12,5 @@
         </xacro:if>
         <geometry>
-          <mesh filename="package://franka_description/meshes/visual/wheel.stl"/>
+          <mesh filename="package://franka_description/meshes/tmr/visual/wheel.stl"/>
         </geometry>
         <material name="darkgrey">
@@ -26,5 +26,5 @@
         </xacro:if>
         <geometry>
-          <mesh filename="package://franka_description/meshes/collision/wheel_simplified.stl"/>
+          <mesh filename="package://franka_description/meshes/tmr/collision/wheel_simplified.stl"/>
         </geometry>
       </collision>

Commit message: fix: update offset values for the torso

File: robots/multi_arm/multi_arm.urdf.xacro (robot description, xacro)
@@ -54,5 +54,5 @@
     <xacro:arg name="torso_kinematics" default="$(find franka_description)/extras/torso_duo/kinematics.yaml"/>
     <xacro:torso name="torso" parent="base_link">
-      <origin xyz="0.20 0 0.30" rpy="0 0 0" />
+      <origin xyz="0.212 0 0.294" rpy="0 0 0" />
     </xacro:torso>
   </xacro:if>
