Commit message: feat: torso visuals added

File: extras/torso_duo/torso.xacro (robot description, xacro)
@@ -6,5 +6,5 @@
       <visual>
         <geometry>
-          <mesh filename="package://franka_description/meshes/torso_duo/collision/torso_collision.stl"/>
+          <mesh filename="package://franka_description/meshes/torso_duo/visual/torso_cover.dae"/>
         </geometry>
         <material name="white">
@@ -14,5 +14,5 @@
       <collision>
         <geometry>
-          <mesh filename="package://franka_description/meshes/torso_duo/collision/torso_collision.stl"/>
+          <mesh filename="package://franka_description/meshes/torso_duo/collision/torso_cover.stl"/>
         </geometry>
       </collision>
