Commit message: fix: lidars inertials updated

File: robots/tmr/nanoscan3/nanoscan3/nanoscan3_macro.xacro (robot description, xacro)
@@ -34,5 +34,7 @@
         <!-- Default inertial for Gazebo - copy and edit block from 'common.xacro'
             to get more realistic behavior -->
-        <xacro:default_inertial/>
+        <xacro:box_inertial x="0.1175" y="0.1006" z="0.05" mass="0.33">
+          <origin xyz="0 0 -0.025" rpy="0 0 0"/>
+        </xacro:box_inertial>
         <visual>
           <geometry>
@@ -76,5 +78,7 @@
       <!-- Default inertial for Gazebo - copy and edit block from 'common.xacro'
            to get more realistic behavior -->
-      <xacro:default_inertial/>
+      <xacro:cylinder_inertial radius="0.43" length="0.03" mass="0.33">
+        <origin xyz="0 0 -0.015" rpy="0 0 0"/>
+      </xacro:cylinder_inertial>
       <visual>
         <!-- These values were determined empirically -->
