Commit message: fix: tmr inertials updated

File: robots/tmr/bogie.xacro (robot description, xacro)
@@ -16,5 +16,7 @@
         </material>
       </visual>
-      <xacro:inertia-box mass="${mass}" width="${width}" depth="${depth}" height="${height}" />
+      <xacro:inertia-box mass="${mass}" width="${width}" depth="${depth}" height="${height}">
+        <origin  rpy="${pi/2} 0 0"/>
+      </xacro:inertia-box>
     </link>
     <joint name="${name}_joint" type="revolute">

File: robots/tmr/caster_wheel.xacro (robot description, xacro)
@@ -4,11 +4,11 @@
   <xacro:macro name="caster_wheel" params="name mass parent length:='0.025' radius:='0.05' caster_joint_z:='-0.074' caster_steering_offset:='-0.035' *origin">
     <xacro:property name="base_width" value="0.04" />
-    <xacro:property name="base_height" value="0.03" />
-    <xacro:property name="base_depth" value="0.003" />
+    <xacro:property name="base_depth" value="0.03" />
+    <xacro:property name="base_height" value="0.003" />
     <link name="${name}_fixed_link" >
       <xacro:macro name="caster_base_geometry" params="xyz:='0 0 0'">
-        <origin xyz="0 0 ${-base_depth/2}" />
+        <origin xyz="0 0 ${-base_height/2}" />
         <geometry>
-          <box size="${base_width} ${base_height} ${base_depth}" />
+          <box size="${base_width} ${base_depth} ${base_height}" />
         </geometry>
         <material name="darkgrey">
@@ -19,5 +19,7 @@
         <xacro:caster_base_geometry/>
       </visual>
-      <xacro:inertia-box mass="${mass}" width="${base_width}" height="${base_height}" depth="${base_depth}" />
+      <xacro:inertia-box mass="${mass}" width="${base_width}" height="${base_height}" depth="${base_depth}">
+        <origin xyz="0 0 ${-base_height/2}" />
+      </xacro:inertia-box>
     </link>
     <joint name="${name}_steering_joint" type="continuous">

File: robots/tmr/inertia.xacro (robot description, xacro)
@@ -23,10 +23,11 @@
   </xacro:macro>
   <!-- According to https://en.wikipedia.org/wiki/List_of_moments_of_inertia#List_of_3D_inertia_tensors -->
-  <xacro:macro name="inertia-box" params="mass width height depth">
+  <xacro:macro name="inertia-box" params="mass width depth height *origin">
     <inertial>
       <mass value="${mass}" />
       <inertia ixx="${1./12 * mass * (height**2 + depth**2)}" ixy="0" ixz="0"
-               iyy="${1./12 * mass * (width**2  + depth**2)}" iyz="0"
-               izz="${1./12 * mass * (width**2  + height**2)}" />
+               iyy="${1./12 * mass * (width**2  + height**2)}" iyz="0"
+               izz="${1./12 * mass * (width**2  + depth**2)}" />
+      <xacro:insert_block name="origin" />
     </inertial>
   </xacro:macro>

File: robots/tmr/tmr.xacro (robot description, xacro)
@@ -21,7 +21,7 @@
     <xacro:property name="caster_bogie_offset" value="0.01" />
     <xacro:property name="platform_height" value="0.3" />
-    <xacro:property name="base_width" value="0.575" />
+    <xacro:property name="base_depth" value="0.575" />
     <xacro:property name="base_height" value="0.294" />
-    <xacro:property name="base_depth" value="0.80" />
+    <xacro:property name="base_width" value="0.80" />
     <xacro:property name="mass" value="75" />
     <xacro:property name="bogie_x" value="-0.18" />
@@ -46,5 +46,5 @@
         <material name="white">
           <color rgba="1.0 1.0 1.0 1.0" />
-        </material>
+        </material>platform_height
       </visual>
       <collision>
@@ -55,7 +55,10 @@
       </collision>
     </link>
+platform_height
     <link name="base_inertia">
       <xacro:inertia-box mass="${mass}" width="${base_width}" height="${base_height}"
-        depth="${base_depth}" />
+        depth="${base_depth}">
+        <origin xyz="0 0 ${platform_height/2} " rpy="0 0 0" />
+      </xacro:inertia-box>
     </link>
     <joint name="base_inertia_joint" type="fixed">
