Commit message: FIX: IMU was not included in the xacro file

File: robots/tmr/tmr.xacro (robot description, xacro)
@@ -13,4 +13,5 @@
     <xacro:include filename="$(find franka_description)/robots/tmr/lidar.xacro" />
     <xacro:include filename="$(find realsense2_description)/urdf/_d455.urdf.xacro" />
+    <xacro:include filename="$(find olv_module_descriptions)/urdf/olv-imu01.urdf.xacro" />
     <xacro:property name="caster_radius" value="0.05" />
     <xacro:property name="caster_mass" value="0.5" />
@@ -131,4 +132,14 @@
       />
     </xacro:if>
+    <!-- IMU -->
+    <link name="imu">
+    </link>
+    <joint name="base_to_imu" type="fixed">
+      <parent link="base_link"/>
+      <child link="imu"/>
+      <origin xyz="-0.176 0.0545 0.15" rpy="0 ${-pi/2} 0"/>
+    </joint>
+    <xacro:olv-imu01 namespace="olv-imu01" parent_link="imu" mounting_side="bottom" mounting_rotation="0">
+    </xacro:olv-imu01>
   </xacro:macro>
 </robot>
