Commit message: feat: ros2 control for tmr v02

File: robots/tmr/tmr.ros2_control.xacro (robot description, xacro)
@@ -21,21 +21,21 @@
         </xacro:if>
       </hardware>
-      <xacro:macro name="configure_joint" params="joint_name initial_position">
+      <xacro:macro name="configure_steering_joint" params="joint_name initial_position">
         <joint name="${joint_name}">
-          <command_interface name="effort" />
-          <command_interface name="velocity" />
           <state_interface name="position">
-            <param name="initial_value">0.0</param>
-          </state_interface>
-          <state_interface name="velocity">
-            <param name="initial_value">0.0</param>
-          </state_interface>
-          <state_interface name="effort">
             <param name="initial_value">0.0</param>
           </state_interface>
         </joint>
       </xacro:macro>
-      <xacro:configure_joint joint_name="${mobile_robot_id}_joint0" initial_position="0.0" />
-      <xacro:configure_joint joint_name="${mobile_robot_id}_joint1" initial_position="0.0" />
+      <xacro:macro name="configure_driving_joint" params="joint_name initial_position">
+        <joint name="${joint_name}">
+          <state_interface name="velocity">
+            <param name="initial_value">0.0</param>
+          </state_interface>
+        </joint>
+      <xacro:configure_steering_joint joint_name="argo_drive_front_steering_joint" initial_position="0.0" />
+      <xacro:configure_driving_joint joint_name="argo_drive_front_joint" initial_position="0.0" />
+      <xacro:configure_steering_joint joint_name="argo_drive_rear_steering_joint" initial_position="0.0" />
+      <xacro:configure_driving_joint joint_name="argo_drive_rear_joint" initial_position="0.0" />
     </ros2_control>
   </xacro:macro>
