Commit message: feat: correct inertials added

File: robots/tmr/argo_drive.xacro (robot description, xacro)
@@ -21,7 +21,15 @@
         <xacro:caster_base_geometry/>
       </visual>
-      <xacro:inertia-box mass="${mass}" width="${base_width}" height="${base_height}" depth="${base_depth}">
-        <origin xyz="0 0 ${-base_height/2}" />
-      </xacro:inertia-box>
+      <inertial>
+        <origin xyz="-0.00019 ${offset_wheel_sign*0.04522} 0.02947" rpy="0 0 0"/>
+        <mass value="11.5"/>
+        <inertia
+          ixx="0.07060497424"
+          ixy="-0.00025482709"
+          ixz="${offset_wheel_sign* (-0.00006283102)}"
+          iyy="0.03433835031"
+          iyz="${offset_wheel_sign*0.00249596715}"
+          izz="0.08926325955"/>
+      </inertial>
     </link>
     <joint name="${name}_fixed_joint" type="fixed">

File: robots/tmr/caster_wheel.xacro (robot description, xacro)
@@ -20,7 +20,15 @@
         <xacro:caster_base_geometry/>
       </visual>
-      <xacro:inertia-box mass="${mass}" width="${base_width}" height="${base_height}" depth="${base_depth}">
-        <origin xyz="0 0 ${-base_height/2}" />
-      </xacro:inertia-box>
+      <inertial>
+        <origin xyz="-0.02365 0.00005 -0.03651" rpy="0 0 0"/>
+        <mass value="0.7"/>
+        <inertia
+          ixx="0.00049538079"
+          ixy="-0.00000042663"
+          ixz="0.00020926011"
+          iyy="0.00070424109"
+          iyz="-0.00000050221"
+          izz="0.00048449394"/>
+      </inertial>
     </link>
     <joint name="${name}_fixed_joint" type="fixed">
@@ -54,5 +62,4 @@
         <xacro:caster_wheel_geometry/>
       </collision>
-      <xacro:inertia-cylinder mass="${mass}" radius="${radius}" h="${length}" />
     </link>
     <joint name="${name}_joint" type="continuous">

File: robots/tmr/rocker_arm.xacro (robot description, xacro)
@@ -16,7 +16,15 @@
         </material>
       </visual>
-      <xacro:inertia-box mass="${mass}" width="${width}" depth="${depth}" height="${height}">
-        <origin  rpy="${pi/2} 0 0"/>
-      </xacro:inertia-box>
+      <inertial>
+        <origin xyz="-0.000344 -0.021232 0.038239" rpy="0 0 0"/>
+        <mass value="5.183973"/>
+        <inertia
+          ixx="0.077004518565"
+          ixy="-0.000040505686"
+          ixz="-0.000026300402"
+          iyy="0.030693821144"
+          iyz="0.002939677599"
+          izz="0.083485865094"/>
+      </inertial>
     </link>
     <joint name="${name}_joint" type="revolute">

File: robots/tmr/tmr.xacro (robot description, xacro)
@@ -48,8 +48,13 @@
     <link name="base_inertia">
       <inertial>
-        <origin xyz="-0.008374 -0.002590 0.160190" rpy="0 0 0"/>
-        <mass value="117.841576"/>
-        <inertia ixx="4.231020518026" ixy="-0.919498121852" ixz="-0.058658325607"
-                iyy="7.057265973509" iyz="-0.004916844299" izz="9.251696036360"/>
+        <origin xyz="0.006619 -0.002210 0.184355" rpy="0 0 0"/>
+        <mass value="88.954183"/>
+        <inertia
+          ixx="3.245524271774"
+          ixy="0.007060314402"
+          ixz="-0.134604220439"
+          iyy="4.162370636125"
+          iyz="-0.010770547630"
+          izz="5.841473351812"/>
       </inertial>
     </link>
