Commit message: feat: reduced kinematic version for tmr v02 added

File: robots/tmr_v02/tmr_v02.urdf.xacro (robot description, xacro)
@@ -9,10 +9,4 @@
   <!-- Define arguments -->
   <xacro:arg name="arm_id" default="tmr_v02" />
-  <!-- Define arguments -->
-  <xacro:arg name="xyz_value" default="0 0 0" />
-  <!-- Define arguments -->
-  <xacro:arg name="rpy_value" default="0 0 0" />
-  <!-- Should self-collision be enabled? -->
-  <xacro:arg name="with_sc" default="false" />
   <!-- Is the robot being controlled with ros2_control?" -->
   <xacro:arg name="ros2_control" default="false" />
@@ -23,12 +17,12 @@
   <!-- Should fake sensors be used? -->
   <xacro:arg name="fake_sensor_commands" default="false" />
-  <!-- Prefixes for arm -->
-  <xacro:arg name="arm_prefix" default="platform" />
+  <!-- Should the reduced kinematic version (without caster wheels) be used? -->
+  <xacro:arg name="reduced_version" default="false" />
   <link name="base">
   </link>
-  <joint name="$(arg arm_prefix)_base" type="fixed">
+  <joint name="base_joint" type="fixed">
     <parent link="base"/>
     <child link="base_link"/>
-    <origin rpy="$(arg rpy_value)" xyz="$(arg xyz_value)"/>
+    <origin rpy="0 0 0" xyz="0 0 0"/>
   </joint>
   <xacro:tmr_v02 mobile_robot_id="$(arg arm_id)"
@@ -36,4 +30,5 @@
               ros2_control="$(arg ros2_control)"
               use_fake_hardware="$(arg use_fake_hardware)"
-              fake_sensor_commands="$(arg fake_sensor_commands)"/>
+              fake_sensor_commands="$(arg fake_sensor_commands)"
+              reduced_version="$(arg reduced_version)"/>
 </robot>

File: robots/tmr_v02/tmr_v02.xacro (robot description, xacro)
@@ -6,5 +6,6 @@
                   ros2_control:=true
                   use_fake_hardware:=false
-                  fake_sensor_commands:=false">
+                  fake_sensor_commands:=false
+                  reduced_version:=false">
     <xacro:include filename="$(find franka_description)/robots/tmr_v02/argo_drive.xacro" />
     <xacro:include filename="$(find franka_description)/robots/tmr_v02/caster_wheel.xacro" />
@@ -65,8 +66,10 @@
     <!-- wheels and suspension -->
     <!-- front -->
-    <xacro:caster_wheel name="caster_front_left" parent="base_link"
-      radius="${caster_radius}">
-      <origin xyz="${caster_x} ${caster_y} ${caster_z}" />
-    </xacro:caster_wheel>
+    <xacro:unless value="${reduced_version}">
+      <xacro:caster_wheel name="caster_front_left" parent="base_link"
+        radius="${caster_radius}">
+        <origin xyz="${caster_x} ${caster_y} ${caster_z}" />
+      </xacro:caster_wheel>
+    </xacro:unless>
     <xacro:argo_drive name="argo_drive_front" parent="base_link" offset_wheel_sign="1"
       radius="${argo_drive_radius}">
@@ -77,9 +80,11 @@
           <origin xyz="${rocker_arm_x} ${rocker_arm_y} ${rocker_arm_z}" />
     </xacro:rocker_arm>
-    <xacro:caster_wheel name="caster_rear_right" parent="rocker_arm_link"
-      radius="${caster_radius}">
-      <origin
-        xyz="${-caster_x - rocker_arm_x} ${-caster_y - rocker_arm_y} ${caster_z - rocker_arm_z}" />
-    </xacro:caster_wheel>
+    <xacro:unless value="${reduced_version}">
+      <xacro:caster_wheel name="caster_rear_right" parent="rocker_arm_link"
+        radius="${caster_radius}">
+        <origin
+          xyz="${-caster_x - rocker_arm_x} ${-caster_y - rocker_arm_y} ${caster_z - rocker_arm_z}" />
+      </xacro:caster_wheel>
+    </xacro:unless>
     <xacro:argo_drive name="argo_drive_rear" parent="rocker_arm_link" offset_wheel_sign="-1"
       radius="${argo_drive_radius}">
