Commit message: fix: collision meshes added to the wheels

File: robots/tmrv0_2/argo_drive.xacro (robot description, xacro)
@@ -9,5 +9,5 @@
     <xacro:property name="mass" value="0.5" />
     <link name="${name}_fixed_link" >
-      <xacro:macro name="caster_base_geometry" params="xyz:='0 0 0'">
+      <xacro:macro name="argo_drive_base_geometry" params="xyz:='0 0 0'">
         <origin xyz="0 ${offset_wheel_sign*(base_depth/2 - offset_wheel)} ${base_height/2 - 0.004}" />
         <geometry>
@@ -19,6 +19,9 @@
       </xacro:macro>
       <visual>
-        <xacro:caster_base_geometry/>
+        <xacro:argo_drive_base_geometry/>
       </visual>
+      <collision>
+        <xacro:argo_drive_base_geometry/>
+      </collision>
       <inertial>
         <origin xyz="-0.00019 ${offset_wheel_sign*0.04522} 0.02947" rpy="0 0 0"/>

File: robots/tmrv0_2/caster_wheel.xacro (robot description, xacro)
@@ -20,4 +20,7 @@
         <xacro:caster_base_geometry/>
       </visual>
+      <collision>
+        <xacro:caster_base_geometry/>
+      </collision>
       <inertial>
         <origin xyz="-0.02365 0.00005 -0.03651" rpy="0 0 0"/>

Commit message: fix: joint names modified for ros2 control

File: robots/tmrv0_2/argo_drive.xacro (robot description, xacro)
@@ -2,5 +2,5 @@
 <robot xmlns:xacro="http://www.ros.org/wiki/xacro" >
   <xacro:include filename="$(find franka_description)/robots/tmrv0_2/inertia.xacro" />
-  <xacro:macro name="argo_drive" params="name parent length:='0.04' radius:='0.05' offset_wheel_sign:='1' *origin">
+  <xacro:macro name="argo_drive" params="name mobile_robot_id parent length:='0.04' radius:='0.05' offset_wheel_sign:='1' *origin">
     <xacro:property name="base_width" value="0.17" />
     <xacro:property name="base_depth" value="0.25" />
@@ -8,4 +8,12 @@
     <xacro:property name="offset_wheel" value="0.085" />
     <xacro:property name="mass" value="0.5" />
+    <xacro:if value="${name == 'argo_drive_front'}">
+      <xacro:property name="steering_joint" value="0" />
+      <xacro:property name="driving_joint" value="1" />
+    </xacro:if>
+    <xacro:if value="${name == 'argo_drive_rear'}">
+      <xacro:property name="steering_joint" value="2" />
+      <xacro:property name="driving_joint" value="3" />
+    </xacro:if>
     <link name="${name}_fixed_link" >
       <xacro:macro name="argo_drive_base_geometry" params="xyz:='0 0 0'">
@@ -42,5 +50,5 @@
     </joint>
     <link name="${name}_steering_link" />
-    <joint name="${name}_steering_joint" type="continuous">
+    <joint name="${mobile_robot_id}_joint_${steering_joint}" type="continuous">
       <origin xyz="0 0 0"/>
       <parent link="${name}_fixed_link" />
@@ -68,5 +76,5 @@
       <xacro:inertia-cylinder mass="${mass}" radius="${radius}" h="${length}" />
     </link>
-    <joint name="${name}_joint" type="continuous">
+    <joint name="${mobile_robot_id}_joint_${driving_joint}" type="continuous">
       <origin xyz ="0 0 0" rpy="0 0 0" />
       <parent link="${name}_steering_link" />

File: robots/tmrv0_2/tmrv0_2.ros2_control.xacro (robot description, xacro)
@@ -21,6 +21,7 @@
         </xacro:if>
       </hardware>
-      <xacro:macro name="configure_steering_joint" params="joint_name initial_position">
+      <xacro:macro name="configure_steering_joint" params="joint_name">
         <joint name="${joint_name}">
+          <command_interface name="position"/>
           <state_interface name="position">
             <param name="initial_value">0.0</param>
@@ -28,14 +29,29 @@
         </joint>
       </xacro:macro>
-      <xacro:macro name="configure_driving_joint" params="joint_name initial_position">
+      <xacro:macro name="configure_driving_joint" params="joint_name">
         <joint name="${joint_name}">
+          <command_interface name="velocity"/>
           <state_interface name="velocity">
             <param name="initial_value">0.0</param>
           </state_interface>
         </joint>
-      <xacro:configure_steering_joint joint_name="argo_drive_front_steering_joint" initial_position="0.0" />
-      <xacro:configure_driving_joint joint_name="argo_drive_front_joint" initial_position="0.0" />
-      <xacro:configure_steering_joint joint_name="argo_drive_rear_steering_joint" initial_position="0.0" />
-      <xacro:configure_driving_joint joint_name="argo_drive_rear_joint" initial_position="0.0" />
+      </xacro:macro>
+      <xacro:configure_steering_joint joint_name="${mobile_robot_id}_joint_0"/>
+      <xacro:configure_driving_joint joint_name="${mobile_robot_id}_joint_1"/>
+      <xacro:configure_steering_joint joint_name="${mobile_robot_id}_joint_2"/>
+      <xacro:configure_driving_joint joint_name="${mobile_robot_id}_joint_3"/>
+      <xacro:macro name="general_purpose_io" params="prefix command_interface index">
+        <gpio name="${prefix}">
+          <command_interface name="${command_interface}"/>
+          <param name="index">${index}</param>
+        </gpio>
+      </xacro:macro>
+      <!-- Cartesian velocity interfaces -->
+      <xacro:general_purpose_io prefix="vx" command_interface="cartesian_velocity" index="0"/>
+      <xacro:general_purpose_io prefix="vy" command_interface="cartesian_velocity" index="1"/>
+      <xacro:general_purpose_io prefix="vz" command_interface="cartesian_velocity" index="2"/>
+      <xacro:general_purpose_io prefix="wx" command_interface="cartesian_velocity" index="3"/>
+      <xacro:general_purpose_io prefix="wy" command_interface="cartesian_velocity" index="4"/>
+      <xacro:general_purpose_io prefix="wz" command_interface="cartesian_velocity" index="5"/>
     </ros2_control>
   </xacro:macro>

File: robots/tmrv0_2/tmrv0_2.xacro (robot description, xacro)
@@ -72,5 +72,5 @@
       </xacro:caster_wheel>
     </xacro:unless>
-    <xacro:argo_drive name="argo_drive_front" parent="base_link" offset_wheel_sign="1"
+    <xacro:argo_drive name="argo_drive_front" mobile_robot_id="${mobile_robot_id}" parent="base_link" offset_wheel_sign="1"
       radius="${argo_drive_radius}">
       <origin xyz="${argo_drive_x} ${-argo_drive_y} ${argo_drive_z}" />
@@ -87,5 +87,5 @@
       </xacro:caster_wheel>
     </xacro:unless>
-    <xacro:argo_drive name="argo_drive_rear" parent="rocker_arm_link" offset_wheel_sign="-1"
+    <xacro:argo_drive name="argo_drive_rear" mobile_robot_id="${mobile_robot_id}" parent="rocker_arm_link" offset_wheel_sign="-1"
       radius="${argo_drive_radius}">
       <origin
