Commit message: feat: mounting points added to tmr

File: robots/tmrv0_2/tmrv0_2.xacro (robot description, xacro)
@@ -135,4 +135,29 @@
       <origin xyz="${-lidar_x} ${-lidar_y} ${lidar_z}" rpy="0 0 0" />
     </joint>
+    <!-- Mounting Points -->
+    <link name="front_mointing_point"/>
+    <joint name="front_mointing_point_joint" type="fixed">
+      <parent link="base_link" />
+      <child link="front_mointing_point" />
+      <origin xyz="0.380705 0.0 0.2345" rpy="${pi} 0 0" />
+    </joint>
+    <link name="rear_mointing_point"/>
+    <joint name="rear_mointing_point_joint" type="fixed">
+      <parent link="base_link" />
+      <child link="rear_mointing_point" />
+      <origin xyz="-0.380705 0.0 0.2345" rpy="${pi} 0 ${pi}" />
+    </joint>
+    <link name="right_mointing_point"/>
+    <joint name="right_mointing_point_joint" type="fixed">
+      <parent link="base_link" />
+      <child link="right_mointing_point" />
+      <origin xyz="0.0 0.272712 0.1145" rpy="${pi} 0 ${pi/2}" />
+    </joint>
+    <link name="left_mointing_point"/>
+    <joint name="left_mointing_point_joint" type="fixed">
+      <parent link="base_link" />
+      <child link="left_mointing_point" />
+      <origin xyz="0.0 -0.272712 0.1145" rpy="${pi} 0 -${pi/2}" />
+    </joint>
     <xacro:if value="${ros2_control}">
       <xacro:include filename="$(find franka_description)/robots/tmrv0_2/tmrv0_2.ros2_control.xacro" />

Commit message: feat: new meshes for the tmr

File: robots/tmrv0_2/tmrv0_2.xacro (robot description, xacro)
@@ -34,5 +34,5 @@
         <origin xyz="0 0 0" rpy="0 0 ${pi}" />
         <geometry>
-          <mesh filename="package://franka_description/meshes/tmrv0_2/visual/tmrv0_2.stl" />
+          <mesh filename="package://franka_description/meshes/tmrv0_2/visual/tmrv0_2.dae" />
         </geometry>
         <material name="white">

Commit message: feat: mobile_fr3_duo added to franka description

File: robots/tmrv0_2/tmrv0_2.xacro (robot description, xacro)
@@ -32,5 +32,5 @@
     <link name="base_link">
       <visual>
-        <origin xyz="0 0 0" rpy="0 0 ${pi}" />
+        <origin xyz="0 0 0" rpy="0 0 0" />
         <geometry>
           <mesh filename="package://franka_description/meshes/tmrv0_2/visual/tmrv0_2.dae" />
@@ -41,5 +41,5 @@
       </visual>
       <collision>
-        <origin xyz="0 0 0" rpy="0 0 ${pi}" />
+        <origin xyz="0 0 0" rpy="0 0 0" />
         <geometry>
           <mesh filename="package://franka_description/meshes/tmrv0_2/collision/tmrv0_2.stl" />
