Commit message: feat: robot_id replaced by robot_type

File: end_effectors/cobot_pump/cobot_pump.urdf.xacro (robot description, xacro)
@@ -5,5 +5,5 @@
   <xacro:include filename="$(find franka_description)/end_effectors/cobot_pump/cobot_pump_arguments.xacro"/>
   <xacro:ee_with_one_link connected_to="$(arg special_connection)"
-                          robot_id="$(arg robot_id)"
+                          robot_type="$(arg robot_type)"
                           ee_id="$(arg ee_id)"
                           ee_inertials="${xacro.load_yaml('$(find franka_description)/end_effectors/$(arg ee_id)/inertials.yaml')}"

File: end_effectors/cobot_pump/cobot_pump_arguments.xacro (robot description, xacro)
@@ -2,5 +2,5 @@
 <robot xmlns:xacro="http://www.ros.org/wiki/xacro">
   <!-- Name for the robot -->
-  <xacro:arg name="robot_id" default="fp3" />
+  <xacro:arg name="robot_type" default="fp3" />
   <!-- End-effector id" -->
   <xacro:arg name="ee_id" default="cobot_pump" />

File: end_effectors/common/ee_with_one_link.xacro (robot description, xacro)
@@ -2,8 +2,8 @@
 <robot xmlns:xacro="http://www.ros.org/wiki/xacro" name="ee_with_one_link">
   <!-- safety_distance: Minimum safety distance in [m] by which the collision volumes are expanded and which is enforced during robot motions -->
-  <xacro:macro name="ee_with_one_link" params="connected_to:='' robot_id arm_prefix:='' ee_id ee_inertials rpy_ee:='0 0 0' xyz_ee:='0 0 0' tcp_xyz:='0 0 0' tcp_rpy:='0 0 0' safety_distance:=0 gazebo:=false description_pkg:=franka_description with_sc:=false">
+  <xacro:macro name="ee_with_one_link" params="connected_to:='' robot_type arm_prefix:='' ee_id ee_inertials rpy_ee:='0 0 0' xyz_ee:='0 0 0' tcp_xyz:='0 0 0' tcp_rpy:='0 0 0' safety_distance:=0 gazebo:=false description_pkg:=franka_description with_sc:=false">
     <xacro:property name="ee_prefix" default="robot_"/>
-    <xacro:unless value="${robot_id == ''}">
-      <xacro:property name="ee_prefix" value="${arm_prefix}${robot_id}_" />
+    <xacro:unless value="${robot_type == ''}">
+      <xacro:property name="ee_prefix" value="${arm_prefix}${robot_type}_" />
     </xacro:unless>
     <xacro:unless value="${connected_to == ''}">

File: end_effectors/common/franka_hand.xacro (robot description, xacro)
@@ -4,5 +4,5 @@
   <xacro:macro name="franka_hand"
                params="connected_to:=''
-                       robot_id arm_prefix:=''
+                       robot_type arm_prefix:=''
                        ee_id ee_inertials
                        rpy_ee:='0 0 0'
@@ -16,6 +16,6 @@
                        no_prefix:=false">
     <xacro:property name="ee_prefix" default="robot_"/>
-    <xacro:unless value="${robot_id == ''}">
-      <xacro:property name="ee_prefix" value="${arm_prefix}${robot_id}_" />
+    <xacro:unless value="${robot_type == ''}">
+      <xacro:property name="ee_prefix" value="${arm_prefix}${robot_type}_" />
     </xacro:unless>
     <xacro:unless value="${connected_to == ''}">

File: end_effectors/franka_hand/franka_hand.urdf.xacro (robot description, xacro)
@@ -5,5 +5,5 @@
   <xacro:include filename="$(find franka_description)/end_effectors/franka_hand/franka_hand_arguments.xacro"/>
   <xacro:franka_hand connected_to="$(arg special_connection)"
-                     robot_id="$(arg robot_id)"
+                     robot_type="$(arg robot_type)"
                      ee_id="$(arg ee_id)_$(arg ee_color)"
                      ee_inertials="${xacro.load_yaml('$(find franka_description)/end_effectors/$(arg ee_id)/inertials.yaml')}"

File: end_effectors/franka_hand/franka_hand_arguments.xacro (robot description, xacro)
@@ -2,5 +2,5 @@
 <robot xmlns:xacro="http://www.ros.org/wiki/xacro">
   <!-- Name for the robot -->
-  <xacro:arg name="robot_id" default="fr3" />
+  <xacro:arg name="robot_type" default="fr3" />
   <!-- End-effector id" -->
   <xacro:arg name="ee_id" default="franka_hand" />

File: robots/common/franka_arm.ros2_control.xacro (robot description, xacro)
@@ -2,5 +2,5 @@
 <robot xmlns:xacro="http://www.ros.org/wiki/xacro">
 <xacro:macro name="franka_arm_ros2_control"
-         params="robot_id
+         params="robot_type
                  robot_ip
                  use_fake_hardware:=false
@@ -14,5 +14,5 @@
         <hardware>
           <param name="version">0.1.0</param>
-          <param name="robot_id">${robot_id}</param>
+          <param name="robot_type">${robot_type}</param>
           <param name="prefix">${arm_prefix}</param>
           <xacro:if value="${use_fake_hardware}">
@@ -51,13 +51,13 @@
         </joint>
       </xacro:macro>
-      <xacro:configure_joint joint_name="${arm_prefix}${robot_id}_joint1" initial_position="0.0"/>
-      <xacro:configure_joint joint_name="${arm_prefix}${robot_id}_joint2" initial_position="${-pi/4}"/>
-      <xacro:configure_joint joint_name="${arm_prefix}${robot_id}_joint3" initial_position="0.0"/>
-      <xacro:configure_joint joint_name="${arm_prefix}${robot_id}_joint4" initial_position="${-3*pi/4}"/>
-      <xacro:configure_joint joint_name="${arm_prefix}${robot_id}_joint5" initial_position="0.0"/>
-      <xacro:configure_joint joint_name="${arm_prefix}${robot_id}_joint6" initial_position="${pi/2}"/>
-      <xacro:configure_joint joint_name="${arm_prefix}${robot_id}_joint7" initial_position="${pi/4}"/>
+      <xacro:configure_joint joint_name="${arm_prefix}${robot_type}_joint1" initial_position="0.0"/>
+      <xacro:configure_joint joint_name="${arm_prefix}${robot_type}_joint2" initial_position="${-pi/4}"/>
+      <xacro:configure_joint joint_name="${arm_prefix}${robot_type}_joint3" initial_position="0.0"/>
+      <xacro:configure_joint joint_name="${arm_prefix}${robot_type}_joint4" initial_position="${-3*pi/4}"/>
+      <xacro:configure_joint joint_name="${arm_prefix}${robot_type}_joint5" initial_position="0.0"/>
+      <xacro:configure_joint joint_name="${arm_prefix}${robot_type}_joint6" initial_position="${pi/2}"/>
+      <xacro:configure_joint joint_name="${arm_prefix}${robot_type}_joint7" initial_position="${pi/4}"/>
       <xacro:if value="${gazebo and hand}">
-        <xacro:configure_joint joint_name="${arm_prefix}${robot_id}_finger_joint1" initial_position="0.0" />
+        <xacro:configure_joint joint_name="${arm_prefix}${robot_type}_finger_joint1" initial_position="0.0" />
       </xacro:if>
       <xacro:macro name="general_purpose_io" params="prefix command_interface index">

File: robots/common/franka_arm.srdf.xacro (robot description, xacro)
@@ -1,6 +1,6 @@
 <?xml version='1.0' encoding='utf-8'?>
 <robot xmlns:xacro="http://www.ros.org/wiki/xacro" >
-    <xacro:macro name="franka_arm_srdf" params="robot_id hand:='true' ee_id:=franka_hand arm_prefix='' no_prefix='false'">
-        <xacro:property name="prefix" value="${'' if no_prefix else arm_prefix + robot_id + '_'}" />
+    <xacro:macro name="franka_arm_srdf" params="robot_type hand:='true' ee_id:=franka_hand arm_prefix='' no_prefix='false'">
+        <xacro:property name="prefix" value="${'' if no_prefix else arm_prefix + robot_type + '_'}" />
         <xacro:include filename="$(find franka_description)/robots/common/group_definition.xacro"/>
         <xacro:property name="tip_link" value="${prefix + 'hand_tcp' if hand and ee_id == 'franka_hand' else prefix + 'link8'}"/>

File: robots/common/franka_arm.xacro (robot description, xacro)
@@ -3,12 +3,12 @@
   <xacro:include filename="$(find franka_description)/robots/common/utils.xacro" />
   <!-- safety_distance: Minimum safety distance in [m] by which the collision volumes are expanded and which is enforced during robot motions -->
-  <!-- robot_id: Namespace of the robot arm. Serves to differentiate between arms in case of multiple instances. -->
+  <!-- robot_type: Namespace of the robot arm. Serves to differentiate between arms in case of multiple instances. -->
   <!-- joint_limits: description of the joint limits that comes from a YAML file. Example definition: ${xacro.load_yaml('$(find franka_description)/robots/fr3/joint_limits.yaml')} -->
   <!-- kinematics: description of the kinematics that comes from a YAML file. Example definition: ${xacro.load_yaml('$(find franka_description)/robots/fr3/kinematics.yaml')} -->
   <!-- inertials: description of the inertials that comes from a YAML file. Example definition: ${xacro.load_yaml('$(find franka_description)/robots/fr3/inertials.yaml')} -->
   <!-- dynamics: description of the dynamics that comes from a YAML file. Example definition: ${xacro.load_yaml('$(find franka_description)/robots/fr3/dynamics.yaml')} -->
-  <xacro:macro name="franka_arm" params="robot_id arm_prefix:='' no_prefix:=false description_pkg:='franka_description' connected_to:='base' xyz:='0 0 0' rpy:='0 0 0' gazebo:='false' safety_distance:=0 joint_limits inertials kinematics accelerometer_config dynamics with_sc:=false" >
-    <!-- Define a property that defaults to 'arm_prefix_robot_id' concatenated with an underscore if 'no_prefix' is not set -->
-    <xacro:property name="prefix" value="${'' if no_prefix else arm_prefix + robot_id + '_'}" />
+  <xacro:macro name="franka_arm" params="robot_type arm_prefix:='' no_prefix:=false description_pkg:='franka_description' connected_to:='base' xyz:='0 0 0' rpy:='0 0 0' gazebo:='false' safety_distance:=0 joint_limits inertials kinematics accelerometer_config dynamics with_sc:=false" >
+    <!-- Define a property that defaults to 'arm_prefix_robot_type' concatenated with an underscore if 'no_prefix' is not set -->
+    <xacro:property name="prefix" value="${'' if no_prefix else arm_prefix + robot_type + '_'}" />
     <xacro:property name="with_accelerometers" value="${'false' if accelerometer_config == 'none' else 'true'}" />
     <xacro:if value="${gazebo}">

File: robots/common/franka_robot.xacro (robot description, xacro)
@@ -2,5 +2,5 @@
 <robot xmlns:xacro="http://www.ros.org/wiki/xacro">
   <xacro:macro name="franka_robot"
-              params="robot_id
+              params="robot_type
                       joint_limits
                       kinematics
@@ -33,5 +33,5 @@
     <xacro:include filename="$(find franka_description)/robots/common/franka_arm.xacro" />
     <xacro:franka_arm
-      robot_id="${robot_id}"
+      robot_type="${robot_type}"
       arm_prefix="${arm_prefix}"
       no_prefix="${no_prefix}"
@@ -51,14 +51,14 @@
       <xacro:include filename="$(find franka_description)/end_effectors/common/franka_hand.xacro"/>
       <xacro:include filename="$(find franka_description)/end_effectors/common/utils.xacro" />
-      <xacro:if value="${robot_id == 'fp3'}">
+      <xacro:if value="${robot_type == 'fp3'}">
         <xacro:property name="ee_color" value="black" />
       </xacro:if>
-      <xacro:if value="${robot_id == 'fr3' or robot_id == 'fer' or robot_id == 'fr3v2' or robot_id == 'fr3v2_1'}">
+      <xacro:if value="${robot_type == 'fr3' or robot_type == 'fer' or robot_type == 'fr3v2' or robot_type == 'fr3v2_1'}">
         <xacro:property name="ee_color" value="white" />
       </xacro:if>
-      <xacro:property name="connection" value="${special_connection if special_connection != '' else robot_id + '_link8'}" />
+      <xacro:property name="connection" value="${special_connection if special_connection != '' else robot_type + '_link8'}" />
       <xacro:franka_hand
         connected_to="${arm_prefix}${connection}"
-        robot_id="${robot_id}"
+        robot_type="${robot_type}"
         arm_prefix="${arm_prefix}"
         ee_id="${ee_id}_${ee_color}"
@@ -77,8 +77,8 @@
       <xacro:include filename="$(find franka_description)/end_effectors/common/ee_with_one_link.xacro"/>
       <xacro:include filename="$(find franka_description)/end_effectors/common/utils.xacro" />
-      <xacro:property name="connection" value="${special_connection if special_connection != '' else robot_id + '_link8'}" />
+      <xacro:property name="connection" value="${special_connection if special_connection != '' else robot_type + '_link8'}" />
       <xacro:ee_with_one_link
         connected_to="${arm_prefix}${connection}"
-        robot_id="${robot_id}"
+        robot_type="${robot_type}"
         arm_prefix="${arm_prefix}"
         ee_id="${ee_id}"
@@ -104,39 +104,39 @@
           <origin xyz="${xyz}" rpy="${rpy}" />
           <parent link="${parent}" />
-          <child  link="${arm_prefix}${robot_id}_link0" />
+          <child  link="${arm_prefix}${robot_type}_link0" />
         </joint>
       </xacro:if>
-      <xacro:gazebo-joint joint="${arm_prefix}${robot_id}_joint1" transmission="hardware_interface/PositionJointInterface" />
-      <xacro:gazebo-joint joint="${arm_prefix}${robot_id}_joint2" transmission="hardware_interface/PositionJointInterface" />
-      <xacro:gazebo-joint joint="${arm_prefix}${robot_id}_joint3" transmission="hardware_interface/PositionJointInterface" />
-      <xacro:gazebo-joint joint="${arm_prefix}${robot_id}_joint4" transmission="hardware_interface/PositionJointInterface" />
-      <xacro:gazebo-joint joint="${arm_prefix}${robot_id}_joint5" transmission="hardware_interface/PositionJointInterface" />
-      <xacro:gazebo-joint joint="${arm_prefix}${robot_id}_joint6" transmission="hardware_interface/PositionJointInterface" />
-      <xacro:gazebo-joint joint="${arm_prefix}${robot_id}_joint7" transmission="hardware_interface/PositionJointInterface" />
-      <xacro:gazebo-joint joint="${arm_prefix}${robot_id}_joint1" transmission="hardware_interface/VelocityJointInterface" />
-      <xacro:gazebo-joint joint="${arm_prefix}${robot_id}_joint2" transmission="hardware_interface/VelocityJointInterface" />
-      <xacro:gazebo-joint joint="${arm_prefix}${robot_id}_joint3" transmission="hardware_interface/VelocityJointInterface" />
-      <xacro:gazebo-joint joint="${arm_prefix}${robot_id}_joint4" transmission="hardware_interface/VelocityJointInterface" />
-      <xacro:gazebo-joint joint="${arm_prefix}${robot_id}_joint5" transmission="hardware_interface/VelocityJointInterface" />
-      <xacro:gazebo-joint joint="${arm_prefix}${robot_id}_joint6" transmission="hardware_interface/VelocityJointInterface" />
-      <xacro:gazebo-joint joint="${arm_prefix}${robot_id}_joint7" transmission="hardware_interface/VelocityJointInterface" />
-      <xacro:gazebo-joint joint="${arm_prefix}${robot_id}_joint1" transmission="hardware_interface/EffortJointInterface" />
-      <xacro:gazebo-joint joint="${arm_prefix}${robot_id}_joint2" transmission="hardware_interface/EffortJointInterface" />
-      <xacro:gazebo-joint joint="${arm_prefix}${robot_id}_joint3" transmission="hardware_interface/EffortJointInterface" />
-      <xacro:gazebo-joint joint="${arm_prefix}${robot_id}_joint4" transmission="hardware_interface/EffortJointInterface" />
-      <xacro:gazebo-joint joint="${arm_prefix}${robot_id}_joint5" transmission="hardware_interface/EffortJointInterface" />
-      <xacro:gazebo-joint joint="${arm_prefix}${robot_id}_joint6" transmission="hardware_interface/EffortJointInterface" />
-      <xacro:gazebo-joint joint="${arm_prefix}${robot_id}_joint7" transmission="hardware_interface/EffortJointInterface" />
-      <xacro:transmission-franka-state robot_id="${robot_id}" />
-      <xacro:transmission-franka-model robot_id="${robot_id}"
-         root="${arm_prefix}${robot_id}_joint1"
-         tip="${arm_prefix}${robot_id}_joint8"
+      <xacro:gazebo-joint joint="${arm_prefix}${robot_type}_joint1" transmission="hardware_interface/PositionJointInterface" />
+      <xacro:gazebo-joint joint="${arm_prefix}${robot_type}_joint2" transmission="hardware_interface/PositionJointInterface" />
+      <xacro:gazebo-joint joint="${arm_prefix}${robot_type}_joint3" transmission="hardware_interface/PositionJointInterface" />
+      <xacro:gazebo-joint joint="${arm_prefix}${robot_type}_joint4" transmission="hardware_interface/PositionJointInterface" />
+      <xacro:gazebo-joint joint="${arm_prefix}${robot_type}_joint5" transmission="hardware_interface/PositionJointInterface" />
+      <xacro:gazebo-joint joint="${arm_prefix}${robot_type}_joint6" transmission="hardware_interface/PositionJointInterface" />
+      <xacro:gazebo-joint joint="${arm_prefix}${robot_type}_joint7" transmission="hardware_interface/PositionJointInterface" />
+      <xacro:gazebo-joint joint="${arm_prefix}${robot_type}_joint1" transmission="hardware_interface/VelocityJointInterface" />
+      <xacro:gazebo-joint joint="${arm_prefix}${robot_type}_joint2" transmission="hardware_interface/VelocityJointInterface" />
+      <xacro:gazebo-joint joint="${arm_prefix}${robot_type}_joint3" transmission="hardware_interface/VelocityJointInterface" />
+      <xacro:gazebo-joint joint="${arm_prefix}${robot_type}_joint4" transmission="hardware_interface/VelocityJointInterface" />
+      <xacro:gazebo-joint joint="${arm_prefix}${robot_type}_joint5" transmission="hardware_interface/VelocityJointInterface" />
+      <xacro:gazebo-joint joint="${arm_prefix}${robot_type}_joint6" transmission="hardware_interface/VelocityJointInterface" />
+      <xacro:gazebo-joint joint="${arm_prefix}${robot_type}_joint7" transmission="hardware_interface/VelocityJointInterface" />
+      <xacro:gazebo-joint joint="${arm_prefix}${robot_type}_joint1" transmission="hardware_interface/EffortJointInterface" />
+      <xacro:gazebo-joint joint="${arm_prefix}${robot_type}_joint2" transmission="hardware_interface/EffortJointInterface" />
+      <xacro:gazebo-joint joint="${arm_prefix}${robot_type}_joint3" transmission="hardware_interface/EffortJointInterface" />
+      <xacro:gazebo-joint joint="${arm_prefix}${robot_type}_joint4" transmission="hardware_interface/EffortJointInterface" />
+      <xacro:gazebo-joint joint="${arm_prefix}${robot_type}_joint5" transmission="hardware_interface/EffortJointInterface" />
+      <xacro:gazebo-joint joint="${arm_prefix}${robot_type}_joint6" transmission="hardware_interface/EffortJointInterface" />
+      <xacro:gazebo-joint joint="${arm_prefix}${robot_type}_joint7" transmission="hardware_interface/EffortJointInterface" />
+      <xacro:transmission-franka-state robot_type="${robot_type}" />
+      <xacro:transmission-franka-model robot_type="${robot_type}"
+         root="${arm_prefix}${robot_type}_joint1"
+         tip="${arm_prefix}${robot_type}_joint8"
        />
       <xacro:if value="${ee_id == 'franka_hand'}">
-        <xacro:gazebo-joint joint="${arm_prefix}${robot_id}_finger_joint1" transmission="hardware_interface/EffortJointInterface" />
-        <xacro:gazebo-joint joint="${arm_prefix}${robot_id}_finger_joint2" transmission="hardware_interface/EffortJointInterface" />
+        <xacro:gazebo-joint joint="${arm_prefix}${robot_type}_finger_joint1" transmission="hardware_interface/EffortJointInterface" />
+        <xacro:gazebo-joint joint="${arm_prefix}${robot_type}_finger_joint2" transmission="hardware_interface/EffortJointInterface" />
         <!-- Friction specific material for Rubber/Rubber contact -->
-        <xacro:gazebo-friction link="${arm_prefix}${robot_id}_leftfinger" mu="1.13" />
-        <xacro:gazebo-friction link="${arm_prefix}${robot_id}_rightfinger" mu="1.13" />
+        <xacro:gazebo-friction link="${arm_prefix}${robot_type}_leftfinger" mu="1.13" />
+        <xacro:gazebo-friction link="${arm_prefix}${robot_type}_rightfinger" mu="1.13" />
       </xacro:if>
     </xacro:if>
@@ -144,5 +144,5 @@
       <xacro:include filename="$(find franka_description)/robots/common/franka_arm.ros2_control.xacro"/>
       <xacro:franka_arm_ros2_control
-          robot_id="${robot_id}"
+          robot_type="${robot_type}"
           robot_ip="${robot_ip}"
           use_fake_hardware="${use_fake_hardware}"
