Commit message: feat: robot_id replaced by robot_type

File: robots/common/utils.xacro (robot description, xacro)
@@ -33,15 +33,15 @@
   <!-- ========================================================== -->
   <xacro:macro name="link_with_sc" params="name no_prefix:='false' rpy:='0 0 0' **self_collision_geometries gazebo:=false with_sc:=false with_accelerometers:=false">
-    <xacro:property name="prefix" value="${'' if no_prefix else arm_prefix + robot_id + '_'}" />
+    <xacro:property name="prefix" value="${'' if no_prefix else arm_prefix + robot_type + '_'}" />
     <!-- sub-link defining detailed meshes for collision with environment -->
     <link name="${prefix}${name}">
       <visual name="${prefix}${name}_visual">
         <geometry>
-          <mesh filename="package://${description_pkg}/meshes/robot_arms/${robot_id}/visual/${name}.dae" />
+          <mesh filename="package://${description_pkg}/meshes/robot_arms/${robot_type}/visual/${name}.dae" />
         </geometry>
       </visual>
       <collision name="${prefix}${name}_collision">
         <geometry>
-          <mesh filename="package://franka_description/meshes/robot_arms/${robot_id}/collision/${name}.stl" />
+          <mesh filename="package://franka_description/meshes/robot_arms/${robot_type}/collision/${name}.stl" />
         </geometry>
       </collision>
@@ -157,23 +157,23 @@
   <!-- when simulating with franka_hw_sim plugin                  -->
   <!--                                                            -->
-  <!-- robot_id - Arm ID of the fer to simulate (default 'fer')     -->
-  <!-- ========================================================== -->
-  <xacro:macro name="transmission-franka-state" params="robot_id:=fer">
-    <transmission name="${arm_prefix}${robot_id}_franka_state">
+  <!-- robot_type - Arm ID of the fer to simulate (default 'fer')     -->
+  <!-- ========================================================== -->
+  <xacro:macro name="transmission-franka-state" params="robot_type:=fer">
+    <transmission name="${arm_prefix}${robot_type}_franka_state">
       <type>franka_hw/FrankaStateInterface</type>
-      <joint name="${arm_prefix}${robot_id}_joint1"><hardwareInterface>franka_hw/FrankaStateInterface</hardwareInterface></joint>
-      <joint name="${arm_prefix}${robot_id}_joint2"><hardwareInterface>franka_hw/FrankaStateInterface</hardwareInterface></joint>
-      <joint name="${arm_prefix}${robot_id}_joint3"><hardwareInterface>franka_hw/FrankaStateInterface</hardwareInterface></joint>
-      <joint name="${arm_prefix}${robot_id}_joint4"><hardwareInterface>franka_hw/FrankaStateInterface</hardwareInterface></joint>
-      <joint name="${arm_prefix}${robot_id}_joint5"><hardwareInterface>franka_hw/FrankaStateInterface</hardwareInterface></joint>
-      <joint name="${arm_prefix}${robot_id}_joint6"><hardwareInterface>franka_hw/FrankaStateInterface</hardwareInterface></joint>
-      <joint name="${arm_prefix}${robot_id}_joint7"><hardwareInterface>franka_hw/FrankaStateInterface</hardwareInterface></joint>
-      <actuator name="${arm_prefix}${robot_id}_motor1"><hardwareInterface>franka_hw/FrankaStateInterface</hardwareInterface></actuator>
-      <actuator name="${arm_prefix}${robot_id}_motor2"><hardwareInterface>franka_hw/FrankaStateInterface</hardwareInterface></actuator>
-      <actuator name="${arm_prefix}${robot_id}_motor3"><hardwareInterface>franka_hw/FrankaStateInterface</hardwareInterface></actuator>
-      <actuator name="${arm_prefix}${robot_id}_motor4"><hardwareInterface>franka_hw/FrankaStateInterface</hardwareInterface></actuator>
-      <actuator name="${arm_prefix}${robot_id}_motor5"><hardwareInterface>franka_hw/FrankaStateInterface</hardwareInterface></actuator>
-      <actuator name="${arm_prefix}${robot_id}_motor6"><hardwareInterface>franka_hw/FrankaStateInterface</hardwareInterface></actuator>
-      <actuator name="${arm_prefix}${robot_id}_motor7"><hardwareInterface>franka_hw/FrankaStateInterface</hardwareInterface></actuator>
+      <joint name="${arm_prefix}${robot_type}_joint1"><hardwareInterface>franka_hw/FrankaStateInterface</hardwareInterface></joint>
+      <joint name="${arm_prefix}${robot_type}_joint2"><hardwareInterface>franka_hw/FrankaStateInterface</hardwareInterface></joint>
+      <joint name="${arm_prefix}${robot_type}_joint3"><hardwareInterface>franka_hw/FrankaStateInterface</hardwareInterface></joint>
+      <joint name="${arm_prefix}${robot_type}_joint4"><hardwareInterface>franka_hw/FrankaStateInterface</hardwareInterface></joint>
+      <joint name="${arm_prefix}${robot_type}_joint5"><hardwareInterface>franka_hw/FrankaStateInterface</hardwareInterface></joint>
+      <joint name="${arm_prefix}${robot_type}_joint6"><hardwareInterface>franka_hw/FrankaStateInterface</hardwareInterface></joint>
+      <joint name="${arm_prefix}${robot_type}_joint7"><hardwareInterface>franka_hw/FrankaStateInterface</hardwareInterface></joint>
+      <actuator name="${arm_prefix}${robot_type}_motor1"><hardwareInterface>franka_hw/FrankaStateInterface</hardwareInterface></actuator>
+      <actuator name="${arm_prefix}${robot_type}_motor2"><hardwareInterface>franka_hw/FrankaStateInterface</hardwareInterface></actuator>
+      <actuator name="${arm_prefix}${robot_type}_motor3"><hardwareInterface>franka_hw/FrankaStateInterface</hardwareInterface></actuator>
+      <actuator name="${arm_prefix}${robot_type}_motor4"><hardwareInterface>franka_hw/FrankaStateInterface</hardwareInterface></actuator>
+      <actuator name="${arm_prefix}${robot_type}_motor5"><hardwareInterface>franka_hw/FrankaStateInterface</hardwareInterface></actuator>
+      <actuator name="${arm_prefix}${robot_type}_motor6"><hardwareInterface>franka_hw/FrankaStateInterface</hardwareInterface></actuator>
+      <actuator name="${arm_prefix}${robot_type}_motor7"><hardwareInterface>franka_hw/FrankaStateInterface</hardwareInterface></actuator>
     </transmission>
   </xacro:macro>
@@ -182,10 +182,10 @@
   <!-- when simulating with franka_hw_sim plugin                    -->
   <!--                                                              -->
-  <!-- robot_id - Arm ID of the fer to simulate (default 'fer')       -->
+  <!-- robot_type - Arm ID of the fer to simulate (default 'fer')       -->
   <!-- root   - Joint name of the base of the robot                 -->
   <!-- tip    - Joint name of the tip of the robot (flange or hand) -->
   <!-- ============================================================ -->
-  <xacro:macro name="transmission-franka-model" params="robot_id:=fer root:=fer_joint1 tip:=fer_joint7">
-    <transmission name="${arm_prefix}${robot_id}_franka_model">
+  <xacro:macro name="transmission-franka-model" params="robot_type:=fer root:=fer_joint1 tip:=fer_joint7">
+    <transmission name="${arm_prefix}${robot_type}_franka_model">
       <type>franka_hw/FrankaModelInterface</type>
       <joint name="${root}">

File: robots/fer/fer.srdf.xacro (robot description, xacro)
@@ -3,5 +3,5 @@
   <xacro:include filename="$(find franka_description)/robots/common/franka_arm.srdf.xacro"/>
   <!-- The ID of the robot model to be used -->
-  <xacro:arg name="robot_id" default="fer" />
+  <xacro:arg name="robot_type" default="fer" />
   <!-- The prefix of the robot -->
   <xacro:arg name="arm_prefix" default="" />
@@ -12,5 +12,5 @@
   <!-- Which end-effector would be mounted at the flange?" -->
   <xacro:arg name="ee_id" default="franka_hand" />
-  <xacro:franka_arm_srdf robot_id="$(arg robot_id)"
+  <xacro:franka_arm_srdf robot_type="$(arg robot_type)"
                       hand="$(arg hand)"
                       ee_id="$(arg ee_id)"

File: robots/fer/fer.urdf.xacro (robot description, xacro)
@@ -4,5 +4,5 @@
   <!-- Define arguments -->
   <!-- The ID of the robot model to be used -->
-  <xacro:arg name="robot_id" default="fer" />
+  <xacro:arg name="robot_type" default="fer" />
   <!-- The prefix of the robot -->
   <xacro:arg name="arm_prefix" default="" />
@@ -44,5 +44,5 @@
   <xacro:property name="prefix" value="$(arg arm_prefix)"/>
   <xacro:property name="modified_prefix" value="${prefix + '_' if prefix else ''}"/>
-  <xacro:franka_robot robot_id="fer"
+  <xacro:franka_robot robot_type="fer"
                       joint_limits="${xacro.load_yaml('$(find franka_description)/robots/fer/joint_limits.yaml')}"
                       inertials="${xacro.load_yaml('$(find franka_description)/robots/fer/inertials.yaml')}"

File: robots/fp3/fp3.srdf.xacro (robot description, xacro)
@@ -3,5 +3,5 @@
   <xacro:include filename="$(find franka_description)/robots/common/franka_arm.srdf.xacro"/>
   <!-- The ID of the robot model to be used -->
-  <xacro:arg name="robot_id" default="fp3" />
+  <xacro:arg name="robot_type" default="fp3" />
   <!-- The prefix of the robot -->
   <xacro:arg name="arm_prefix" default="" />
@@ -12,5 +12,5 @@
   <!-- Which end-effector would be mounted at the flange?" -->
   <xacro:arg name="ee_id" default="franka_hand" />
-  <xacro:franka_arm_srdf robot_id="$(arg robot_id)"
+  <xacro:franka_arm_srdf robot_type="$(arg robot_type)"
                       hand="$(arg hand)"
                       ee_id="$(arg ee_id)"

File: robots/fp3/fp3.urdf.xacro (robot description, xacro)
@@ -4,5 +4,5 @@
   <!-- Define arguments -->
   <!-- The ID of the robot model to be used -->
-  <xacro:arg name="robot_id" default="fp3" />
+  <xacro:arg name="robot_type" default="fp3" />
   <!-- The prefix of the robot -->
   <xacro:arg name="arm_prefix" default="" />
@@ -44,5 +44,5 @@
   <xacro:property name="prefix" value="$(arg arm_prefix)"/>
   <xacro:property name="modified_prefix" value="${prefix + '_' if prefix else ''}"/>
-  <xacro:franka_robot robot_id="fp3"
+  <xacro:franka_robot robot_type="fp3"
                       joint_limits="${xacro.load_yaml('$(find franka_description)/robots/fp3/joint_limits.yaml')}"
                       inertials="${xacro.load_yaml('$(find franka_description)/robots/fp3/inertials.yaml')}"

File: robots/fr3/fr3.srdf.xacro (robot description, xacro)
@@ -3,5 +3,5 @@
   <xacro:include filename="$(find franka_description)/robots/common/franka_arm.srdf.xacro"/>
   <!-- The ID of the robot model to be used -->
-  <xacro:arg name="robot_id" default="fr3" />
+  <xacro:arg name="robot_type" default="fr3" />
   <!-- The prefix of the robot -->
   <xacro:arg name="arm_prefix" default="" />
@@ -12,5 +12,5 @@
   <!-- Which end-effector would be mounted at the flange?" -->
   <xacro:arg name="ee_id" default="franka_hand" />
-  <xacro:franka_arm_srdf robot_id="$(arg robot_id)"
+  <xacro:franka_arm_srdf robot_type="$(arg robot_type)"
                       hand="$(arg hand)"
                       ee_id="$(arg ee_id)"

File: robots/fr3/fr3.urdf.xacro (robot description, xacro)
@@ -4,5 +4,5 @@
   <!-- Define arguments -->
   <!-- The ID of the robot model to be used -->
-  <xacro:arg name="robot_id" default="fr3" />
+  <xacro:arg name="robot_type" default="fr3" />
   <!-- The prefix of the robot -->
   <xacro:arg name="arm_prefix" default="" />
@@ -44,5 +44,5 @@
   <xacro:property name="prefix" value="$(arg arm_prefix)"/>
   <xacro:property name="modified_prefix" value="${prefix + '_' if prefix else ''}"/>
-  <xacro:franka_robot robot_id="fr3"
+  <xacro:franka_robot robot_type="fr3"
                       joint_limits="${xacro.load_yaml('$(find franka_description)/robots/fr3/joint_limits.yaml')}"
                       inertials="${xacro.load_yaml('$(find franka_description)/robots/fr3/inertials.yaml')}"

File: robots/fr3_duo/fr3_duo.urdf.xacro (robot description, xacro)
@@ -5,6 +5,6 @@
   <!-- Define arguments -->
   <!-- The IDs of the robot models to be used -->
-  <xacro:arg name="robot_ids" default="['fr3v2','fr3v2']" />
-  <xacro:property name="robot_ids_list" value="${$(arg robot_ids)}" />
+  <xacro:arg name="robot_types" default="['fr3v2','fr3v2']" />
+  <xacro:property name="robot_types_list" value="${$(arg robot_types)}" />
   <!-- Don't print a prefix for joints, visuals, and links? -->
   <xacro:arg name="no_prefix" default="false"/>
@@ -66,11 +66,11 @@
         <origin rpy="${mount_corner.kinematic.roll} ${mount_corner.kinematic.pitch} ${mount_corner.kinematic.yaw}" xyz="${mount_corner.kinematic.x} ${mount_corner.kinematic.y} ${mount_corner.kinematic.z}"/>
       </joint>
-      <xacro:property name="robot_id_i" value="${robot_ids_list[i]}"/>
-      <xacro:arg name="inertials_path" default="$(find franka_description)/robots/${robot_id_i}/inertials.yaml"/>
-      <xacro:arg name="kinematics_path" default="$(find franka_description)/robots/${robot_id_i}/kinematics.yaml"/>
-      <xacro:arg name="dynamics_path" default="$(find franka_description)/robots/${robot_id_i}/dynamics.yaml"/>
-      <xacro:arg name="joint_limits_path" default="$(find franka_description)/robots/${robot_id_i}/joint_limits.yaml"/>
-      <xacro:arg name="accelerometers_path" default="$(find franka_description)/robots/${robot_id_i}/accelerometers.yaml"/>
-      <xacro:franka_robot robot_id="${robot_id_i}"
+      <xacro:property name="robot_type_i" value="${robot_types_list[i]}"/>
+      <xacro:arg name="inertials_path" default="$(find franka_description)/robots/${robot_type_i}/inertials.yaml"/>
+      <xacro:arg name="kinematics_path" default="$(find franka_description)/robots/${robot_type_i}/kinematics.yaml"/>
+      <xacro:arg name="dynamics_path" default="$(find franka_description)/robots/${robot_type_i}/dynamics.yaml"/>
+      <xacro:arg name="joint_limits_path" default="$(find franka_description)/robots/${robot_type_i}/joint_limits.yaml"/>
+      <xacro:arg name="accelerometers_path" default="$(find franka_description)/robots/${robot_type_i}/accelerometers.yaml"/>
+      <xacro:franka_robot robot_type="${robot_type_i}"
                           joint_limits="${xacro.load_yaml('$(arg joint_limits_path)')}"
                           inertials="${xacro.load_yaml('$(arg inertials_path)')}"

File: robots/fr3_duo/fr3_duo_arm.urdf.xacro (robot description, xacro)
@@ -5,5 +5,5 @@
   <!-- Define arguments -->
   <!-- The ID of the robot model to be used -->
-  <xacro:arg name="robot_id" default="fr3v2" />
+  <xacro:arg name="robot_type" default="fr3v2" />
   <!-- The prefix of the robot -->
   <xacro:arg name="arm_prefix" default="" />
@@ -49,5 +49,5 @@
   <xacro:arg name="mount_kinematics" default="$(find franka_description)/robots/fr3_duo/fr3_duo_mount/kinematics.yaml"/>
   <xacro:property name="mount_to_base" value="${xacro.load_yaml('$(arg mount_kinematics)')}"/>
-  <xacro:property name="robot_id_i" value="$(arg robot_id)"/>
+  <xacro:property name="robot_type_i" value="$(arg robot_type)"/>
   <xacro:property name="arm_prefix_i" value="$(arg arm_prefix)"/>
   <joint name="${arm_prefix_i}_base_joint" type="fixed">
@@ -62,10 +62,10 @@
     <origin rpy="${mount_corner.kinematic.roll} ${mount_corner.kinematic.pitch} ${mount_corner.kinematic.yaw}" xyz="${mount_corner.kinematic.x} ${mount_corner.kinematic.y} ${mount_corner.kinematic.z}"/>
   </joint>
-  <xacro:arg name="inertials_path" default="$(find franka_description)/robots/${robot_id_i}/inertials.yaml"/>
-  <xacro:arg name="kinematics_path" default="$(find franka_description)/robots/${robot_id_i}/kinematics.yaml"/>
-  <xacro:arg name="accelerometers_path" default="$(find franka_description)/robots/${robot_id_i}/accelerometers.yaml"/>
-  <xacro:arg name="dynamics_path" default="$(find franka_description)/robots/${robot_id_i}/dynamics.yaml"/>
-  <xacro:arg name="joint_limits_path" default="$(find franka_description)/robots/${robot_id_i}/joint_limits.yaml"/>
-  <xacro:franka_robot robot_id="${robot_id_i}"
+  <xacro:arg name="inertials_path" default="$(find franka_description)/robots/${robot_type_i}/inertials.yaml"/>
+  <xacro:arg name="kinematics_path" default="$(find franka_description)/robots/${robot_type_i}/kinematics.yaml"/>
+  <xacro:arg name="accelerometers_path" default="$(find franka_description)/robots/${robot_type_i}/accelerometers.yaml"/>
+  <xacro:arg name="dynamics_path" default="$(find franka_description)/robots/${robot_type_i}/dynamics.yaml"/>
+  <xacro:arg name="joint_limits_path" default="$(find franka_description)/robots/${robot_type_i}/joint_limits.yaml"/>
+  <xacro:franka_robot robot_type="${robot_type_i}"
                       joint_limits="${xacro.load_yaml('$(arg joint_limits_path)')}"
                       inertials="${xacro.load_yaml('$(arg inertials_path)')}"

File: robots/fr3v2/fr3v2.srdf.xacro (robot description, xacro)
@@ -3,5 +3,5 @@
   <xacro:include filename="$(find franka_description)/robots/common/franka_arm.srdf.xacro"/>
   <!-- The ID of the robot model to be used -->
-  <xacro:arg name="robot_id" default="fr3v2" />
+  <xacro:arg name="robot_type" default="fr3v2" />
   <!-- The prefix of the robot -->
   <xacro:arg name="arm_prefix" default="" />
@@ -12,5 +12,5 @@
   <!-- Which end-effector would be mounted at the flange?" -->
   <xacro:arg name="ee_id" default="franka_hand" />
-  <xacro:franka_arm_srdf robot_id="$(arg robot_id)"
+  <xacro:franka_arm_srdf robot_type="$(arg robot_type)"
                       hand="$(arg hand)"
                       ee_id="$(arg ee_id)"
